Commit message: sapve-pickle

File: ldr-harambe/robot_harambe.urdf (robot description, URDF)
Before this commit: robot robot_harambe, 26 links, 23 joints
Links:
- link ankle_assembly: geometry collision mesh filename=package://assets/ankle_ear.stl; collision mesh filename=package://assets/ankle_shaft.stl
- link ankle_assembly_2: geometry collision mesh filename=package://assets/ankle_ear.stl; collision mesh filename=package://assets/ankle_shaft.stl
- link ankle_assembly_3: geometry collision mesh filename=package://assets/ankle_ear.stl; collision mesh filename=package://assets/ankle_shaft.stl
- link ankle_assembly_4: geometry collision mesh filename=package://assets/ankle_ear.stl; collision mesh filename=package://assets/ankle_shaft.stl
- link urdf_base: geometry collision mesh filename=package://assets/b_base.stl; collision mesh filename=package://assets/f_base.stl
- link urdf_hip_assembly: geometry collision mesh filename=package://assets/hip.stl; collision mesh filename=package://assets/stator_x8_p20_120_unified.stl
- link urdf_hip_assembly_2: geometry collision mesh filename=package://assets/hip.stl; collision mesh filename=package://assets/stator_x8_p20_120_unified.stl
- link urdf_l_elbow_assembly: geometry collision mesh filename=package://assets/elbow_limiter.stl; collision mesh filename=package://assets/l_elbow.stl
- link urdf_l_lower_forearm_assembly: geometry collision mesh filename=package://assets/hand_limiter.stl; collision mesh filename=package://assets/l_lower_forearm.stl
- link urdf_l_shoulder_assembly: geometry collision mesh filename=package://assets/l_shoulder.stl; collision mesh filename=package://assets/stator_x6_p20_60_unified.stl
- link urdf_l_tibia_assembly: geometry collision mesh filename=package://assets/12_7mm_ball_with_6mm_hole.stl; collision mesh filename=package://assets/12_7mm_ball_with_6mm_hole.stl
- link urdf_l_upper_arm_assembly: geometry collision mesh filename=package://assets/arm_limiter.stl; collision mesh filename=package://assets/l_upper_arm.stl
- link urdf_l_upper_femur_assembly: geometry collision mesh filename=package://assets/l_upper_femur.stl; collision mesh filename=package://assets/rotor_x8_p20_120.stl
- link urdf_l_upper_forearm_assembly: geometry collision mesh filename=package://assets/forearm_limiter.stl; collision mesh filename=package://assets/l_upper_forearm.stl
- link urdf_l_wrist_assembly: geometry collision mesh filename=package://assets/l_hand.stl; collision mesh filename=package://assets/l_wrist.stl
- link urdf_lower_femur_assembly: geometry collision mesh filename=package://assets/lower_femur.stl; collision mesh filename=package://assets/stator_x8_p20_120_unified.stl
- link urdf_lower_femur_assembly_2: geometry collision mesh filename=package://assets/lower_femur.stl; collision mesh filename=package://assets/stator_x8_p20_120_unified.stl
- link urdf_r_elbow_assembly: geometry collision mesh filename=package://assets/r_elbow.stl; collision mesh filename=package://assets/stator_x6_p20_60_unified.stl
- link urdf_r_lower_forearm_assembly: geometry collision mesh filename=package://assets/r_lower_forearm.stl; collision mesh filename=package://assets/stator_x4_p36_36_unified.stl
- link urdf_r_shoulder_assembly: geometry collision mesh filename=package://assets/r_shoulder.stl; collision mesh filename=package://assets/stator_x6_p20_60_unified.stl
- link urdf_r_tibia_assembly: geometry collision mesh filename=package://assets/12_7mm_ball_with_6mm_hole.stl; collision mesh filename=package://assets/12_7mm_ball_with_6mm_hole.stl
- link urdf_r_upper_arm_assembly: geometry collision mesh filename=package://assets/r_upper_arm.stl; collision mesh filename=package://assets/stator_x4_p36_36_unified.stl
- link urdf_r_upper_femur_assemby: geometry collision mesh filename=package://assets/r_upper_femur.stl; collision mesh filename=package://assets/stator_x8_p20_120_unified.stl
- link urdf_r_upper_forearm_assembly: geometry collision mesh filename=package://assets/r_upper_forearm.stl; collision mesh filename=package://assets/stator_x4_p36_36_unified.stl
- link urdf_r_wrist_assembly: geometry collision mesh filename=package://assets/r_hand.stl; collision mesh filename=package://assets/r_wrist.stl
- link urdf_simplified_torso_sub_assembly: geometry collision mesh filename=package://assets/back_access.stl; collision mesh filename=package://assets/head.stl

Commit message: mujoco CoM

File: ldr-harambe/robot_harambe.urdf (robot description, URDF)
Before this commit: robot robot_harambe, 26 links, 23 joints
Joints:
- added joint left_ankle_pitch_joint_2: type fixed, parent urdf_l_tibia_assembly, child ankle_assembly_2, origin xyz=-0 -0.395 0.03 rpy=-3.14159 0 0
- added joint right_ankle_pitch_joint_2: type fixed, parent urdf_r_tibia_assembly, child ankle_assembly_4, origin xyz=0.025 0.423 0.056 rpy=-3.14159 1.5708 0
- joint left_ankle_pitch_joint: child ankle_assembly_2 -> ankle_assembly
- joint right_ankle_pitch_joint: child ankle_assembly_4 -> ankle_assembly_3

Commit message: harambe v0.3 export

File: ldr-harambe/robot_harambe.urdf (robot description, URDF)
Before this commit: robot robot_harambe, 26 links, 25 joints
Links:
- removed link ankle_assembly
- removed link ankle_assembly_2
- removed link ankle_assembly_3
- removed link ankle_assembly_4
- removed link urdf_simplified_torso_sub_assembly
- added link udrf_ankle_assembly, mass 0.0818219; collision mesh filename=package://assets/udrf_ankle_assembly.stl; visual mesh filename=package://assets/udrf_ankle_assembly.stl
- added link udrf_ankle_assembly_2, mass 0.0818219; collision mesh filename=package://assets/udrf_ankle_assembly.stl; visual mesh filename=package://assets/udrf_ankle_assembly.stl
- added link urdf_foot_assembly, mass 0.504; collision mesh filename=package://assets/urdf_foot_assembly.stl; visual mesh filename=package://assets/urdf_foot_assembly.stl
- added link urdf_foot_assembly_2, mass 0.504; collision mesh filename=package://assets/urdf_foot_assembly.stl; visual mesh filename=package://assets/urdf_foot_assembly.stl
- added link urdf_simplified_torso, mass 5.9; collision mesh filename=package://assets/back_access.stl; collision mesh filename=package://assets/head.stl
- link urdf_l_elbow_assembly: mass 2.98735 -> 1.109; geometry collision mesh filename=package://assets/stator_x6_p20_60_unified.stl; collision mesh filename=package://assets/urdf_l_elbow_simplified.stl
- link urdf_l_lower_forearm_assembly: mass 0.553 -> 0.618; geometry collision mesh filename=package://assets/stator_x4_p36_36_unified.stl; collision mesh filename=package://assets/urdf_l_lower_forearm_simplified.stl
- link urdf_l_shoulder_assembly: mass 3.07135 -> 1.246
- link urdf_l_tibia_assembly: mass 4.89318 -> 6.45981; geometry collision mesh filename=package://assets/m6_threaded_bar_225mm.stl; collision mesh filename=package://assets/m6_threaded_bar_300mm.stl
- link urdf_l_upper_arm_assembly: mass 0.822 -> 0.802; geometry collision mesh filename=package://assets/stator_x4_p36_36_unified.stl; collision mesh filename=package://assets/urdf_l_upper_arm_simplified.stl
- link urdf_l_upper_femur_assembly: geometry collision mesh filename=package://assets/l_upper_femur.stl; collision mesh filename=package://assets/stator_x8_p20_120_unified.stl
- link urdf_l_upper_forearm_assembly: mass 0.727 -> 0.707; geometry collision mesh filename=package://assets/stator_x4_p36_36_unified.stl; collision mesh filename=package://assets/urdf_l_upper_forearm_simplified.stl
- link urdf_r_elbow_assembly: mass 2.93435 -> 1.109
- link urdf_r_shoulder_assembly: mass 2.84535 -> 1.02
- link urdf_r_tibia_assembly: mass 3.4106 -> 6.45984; geometry collision mesh filename=package://assets/m6_threaded_bar_225mm.stl; collision mesh filename=package://assets/m6_threaded_bar_300mm.stl
Joints:
- removed joint left_ankle_pitch_joint_2
- removed joint right_ankle_pitch_joint_2
- added joint left_ankle_roll_joint: type revolute, parent udrf_ankle_assembly, child urdf_foot_assembly, origin xyz=-0.012 0.028 -0.004 rpy=0 1.5708 0, axis 0 0 1, limit lower=-0.785398 upper=0.785398 effort=10 velocity=10
- added joint right_ankle_roll_joint: type revolute, parent urdf_r_tibia_assembly, child udrf_ankle_assembly_2, origin xyz=0 0.395 0.059 rpy=0 -0 0, axis 0 0 1, limit lower=-0.785398 upper=0.785398 effort=10 velocity=10
- joint left_ankle_pitch_joint: child ankle_assembly -> udrf_ankle_assembly; origin xyz=-0 -0.395 0.03 rpy=-3.14159 0 0 -> xyz=-0 0.395 -0.051 rpy=0 -0 0
- joint left_elbow_pitch_joint_X6: origin xyz=-0.04 0 -0.065 rpy=1.5708 0 1.5708 -> xyz=-0 -0.035 -0.075 rpy=-1.5708 1.5708 0
- joint left_hip_pitch_joint: limit lower=-1.5708 upper=2.53073 effort=10 velocity=10 -> lower=-2.53073 upper=1.5708 effort=10 velocity=10; origin xyz=-0.111301 0.0333787 -0.467748 rpy=1.5708 0 1.5708 -> xyz=-0.111301 0.0333787 -0.467748 rpy=-1.5708 -0 1.5708
- joint left_hip_roll_joint: limit lower=-3.14159 upper=0.349066 effort=10 velocity=10 -> lower=-0.349066 upper=3.14159 effort=10 velocity=10; origin xyz=0.055 0 -0.073 rpy=-0 -1.5708 0 -> xyz=0.055 0 0.073 rpy=-0 1.5708 0
- joint left_hip_yaw_joint: origin xyz=-0 -0.217 0.053 rpy=-1.5708 0 -0 -> xyz=-0 0.217 -0.053 rpy=-1.5708 0 0
- joint left_knee_joint: limit lower=0 upper=1.5708 effort=10 velocity=10 -> lower=-0.174533 upper=1.5708 effort=10 velocity=10; origin xyz=-0.055 -0 -0.113 rpy=1.5708 0 1.5708 -> xyz=-0.055 -0 0.113 rpy=1.5708 0 -1.5708
- joint left_shoulder_pitch_joint_X6: limit lower=-1.5708 upper=3.14159 effort=10 velocity=10 -> lower=-3.14159 upper=1.5708 effort=10 velocity=10; origin xyz=-0.169498 -4.00839e-06 -0.427 rpy=-1.5708 0 -1.5708 -> xyz=-0.1755 -5.1e-11 0.423977 rpy=-1.5708 0 1.5708; parent urdf_simplified_torso_sub_assembly -> urdf_simplified_torso
- joint left_shoulder_roll_joint_X6: origin xyz=0.036 0 -0.07 rpy=-3.14159 -1.5708 0 -> xyz=0.046 -0 0.07 rpy=-0 1.5708 0
- joint left_shoulder_yaw_joint_X4: origin xyz=0 0.17 -0.046 rpy=1.5708 -0 -0 -> xyz=-0 0.165 -0.046 rpy=1.5708 1.5708 0
- joint left_wrist_roll_joint_X4: origin xyz=0 0.033 -0.0565 rpy=1.5708 0 -0 -> xyz=0 0.027 -0.0615 rpy=-1.5708 -0 0
- joint left_wrist_yaw_joint_X4: origin xyz=-0 -0.168 0.04 rpy=-1.5708 -1.5708 0 -> xyz=0.163 0 0.035 rpy=0 -1.5708 0
- joint right_ankle_pitch_joint: child ankle_assembly_3 -> urdf_foot_assembly_2; origin xyz=0.025 0.423 0.056 rpy=-3.14159 1.5708 0 -> xyz=-0.012 0.028 -0.004 rpy=0 1.5708 0; parent urdf_r_tibia_assembly -> udrf_ankle_assembly_2
- joint right_elbow_pitch_joint_X6: origin xyz=0.04 -0 -0.065 rpy=-1.5708 -0 1.5708 -> xyz=0.04 0 -0.065 rpy=-1.5708 0 1.5708
- joint right_hip_pitch_joint: limit lower=-2.51486 upper=1.58667 effort=10 velocity=10 -> lower=-2.53073 upper=1.5708 effort=10 velocity=10; origin xyz=0.107699 0.0333787 -0.467748 rpy=-1.5708 -0 1.5708 -> xyz=0.107699 0.0333787 -0.467748 rpy=1.5708 -0 1.5708
- joint right_hip_roll_joint: limit lower=-0.35061 upper=3.14005 effort=10 velocity=10 -> lower=-3.14159 upper=0.349066 effort=10 velocity=10; origin xyz=0.0549931 -0.000872784 -0.078 rpy=1.5708 1.56925 -1.58667 -> xyz=0.055 0 0.078 rpy=-3.14159 -1.5708 0
- joint right_hip_yaw_joint: limit lower=-1.57082 upper=1.57077 effort=10 velocity=10 -> lower=-1.5708 upper=1.5708 effort=10 velocity=10; origin xyz=-0 -0.217 0.053 rpy=-1.5708 0 0 -> xyz=0 0.217 -0.053 rpy=-1.5708 0 -0
- joint right_knee_joint: limit lower=-0.191906 upper=2.33882 effort=10 velocity=10 -> lower=-0.174533 upper=1.5708 effort=10 velocity=10; origin xyz=0.055 1.37102e-06 -0.113 rpy=-1.5708 0.0173732 1.57082 -> xyz=0.055 -0 0.113 rpy=1.5708 0 -1.5708
- joint right_shoulder_pitch_joint_X6: origin xyz=0.181502 -4.00839e-06 -0.427 rpy=1.5708 0 -1.5708 -> xyz=0.1755 -5.1e-11 0.423977 rpy=-1.5708 -0 1.5708; parent urdf_simplified_torso_sub_assembly -> urdf_simplified_torso
- joint right_shoulder_roll_joint_X6: limit lower=0 upper=3.14159 effort=10 velocity=10 -> lower=-3.14159 upper=0 effort=10 velocity=10
- joint right_shoulder_yaw_joint_X4: origin xyz=0 -0.17 0.041 rpy=-1.5708 -0 0 -> xyz=0 -0.17 0.041 rpy=-1.5708 0 0
- joint right_wrist_roll_joint_X4: origin xyz=-0 0.033 -0.0565 rpy=1.5708 -0 -0 -> xyz=-0 -0.027 0.0565 rpy=1.5708 0 -0
- joint right_wrist_yaw_joint_X4: origin xyz=0 0.168 0.04 rpy=1.5708 1.5708 0 -> xyz=-0 0.168 0.04 rpy=-1.5708 1.5708 0
- joint waist_yaw_joint: child urdf_simplified_torso_sub_assembly -> urdf_simplified_torso; origin xyz=0.000698852 0.0333787 -0.300748 rpy=3.14159 -0 0 -> xyz=0.000698852 0.0333787 -0.300748 rpy=0 -0 0
