Commit message: joints limits from actuators specs

File: ldr-harambe-v0.3-procesed/robot_harambe_v03_fixed_axes_limits.urdf (robot description, URDF)
Before this commit: robot robot_harambe_v0.3, 26 links, 25 joints
Joints:
- joint left_ankle_pitch_joint: limit lower=-0.79 upper=0.79 effort=100 velocity=100 -> lower=-0.79 upper=0.79 effort=43 velocity=13.3
- joint left_ankle_roll_joint: limit lower=-0.79 upper=0.79 effort=100 velocity=100 -> lower=-0.79 upper=0.79 effort=43 velocity=13.3
- joint left_elbow_pitch_joint_X6: limit lower=-1.31 upper=1.83 effort=100 velocity=100 -> lower=-1.31 upper=1.83 effort=20 velocity=16.02
- joint left_hip_pitch_joint: limit lower=-2.53 upper=1.57 effort=100 velocity=100 -> lower=-2.53 upper=1.57 effort=43 velocity=13.3
- joint left_hip_roll_joint: limit lower=-0.35 upper=3.14 effort=100 velocity=100 -> lower=-0.35 upper=3.14 effort=43 velocity=13.3
- joint left_hip_yaw_joint: limit lower=-1.57 upper=1.57 effort=100 velocity=100 -> lower=-1.57 upper=1.57 effort=43 velocity=13.3
- joint left_knee_joint: limit lower=-0.17 upper=1.57 effort=100 velocity=100 -> lower=-0.17 upper=1.57 effort=43 velocity=13.3
- joint left_shoulder_pitch_joint_X6: limit lower=-3.02 upper=1.69 effort=100 velocity=100 -> lower=-3.02 upper=1.69 effort=20 velocity=16.02
- joint left_shoulder_roll_joint_X6: limit lower=-0.21 upper=2.93 effort=100 velocity=100 -> lower=-0.21 upper=2.93 effort=20 velocity=16.02
- joint left_shoulder_yaw_joint_X4: limit lower=-1.75 upper=2.97 effort=100 velocity=100 -> lower=-1.75 upper=2.97 effort=10.5 velocity=8.69
- joint left_wrist_roll_joint_X4: limit lower=-1.57 upper=1.57 effort=100 velocity=100 -> lower=-1.57 upper=1.57 effort=10.5 velocity=8.69
- joint left_wrist_yaw_joint_X4: limit lower=-2.36 upper=2.36 effort=100 velocity=100 -> lower=-2.36 upper=2.36 effort=10.5 velocity=8.69
- joint right_ankle_pitch_joint: limit lower=-0.79 upper=0.79 effort=100 velocity=100 -> lower=-0.79 upper=0.79 effort=43 velocity=13.3
- joint right_ankle_roll_joint: limit lower=-0.79 upper=0.79 effort=100 velocity=100 -> lower=-0.79 upper=0.79 effort=43 velocity=13.3
- joint right_elbow_pitch_joint_X6: limit lower=-1.31 upper=1.83 effort=100 velocity=100 -> lower=-1.31 upper=1.83 effort=20 velocity=16.02
- joint right_hip_pitch_joint: limit lower=-2.53 upper=1.57 effort=100 velocity=100 -> lower=-2.53 upper=1.57 effort=43 velocity=13.3
- joint right_hip_roll_joint: limit lower=-3.14 upper=0.35 effort=100 velocity=100 -> lower=-3.14 upper=0.35 effort=43 velocity=13.3
- joint right_hip_yaw_joint: limit lower=-1.57 upper=1.57 effort=100 velocity=100 -> lower=-1.57 upper=1.57 effort=43 velocity=13.3
- joint right_knee_joint: limit lower=-0.17 upper=1.57 effort=100 velocity=100 -> lower=-0.17 upper=1.57 effort=43 velocity=13.3
- joint right_shoulder_pitch_joint_X6: limit lower=-3.02 upper=1.69 effort=100 velocity=100 -> lower=-3.02 upper=1.69 effort=20 velocity=16.02
- joint right_shoulder_roll_joint_X6: limit lower=-2.93 upper=0.21 effort=100 velocity=100 -> lower=-2.93 upper=0.21 effort=20 velocity=16.02
- joint right_shoulder_yaw_joint_X4: limit lower=-2.97 upper=1.75 effort=100 velocity=100 -> lower=-2.97 upper=1.75 effort=10.5 velocity=8.69
- joint right_wrist_roll_joint_X4: limit lower=-1.57 upper=1.57 effort=100 velocity=100 -> lower=-1.57 upper=1.57 effort=10.5 velocity=8.69
- joint right_wrist_yaw_joint_X4: limit lower=-2.36 upper=2.36 effort=100 velocity=100 -> lower=-2.36 upper=2.36 effort=10.5 velocity=8.69
- joint waist_yaw_joint: limit lower=-1.57 upper=1.57 effort=100 velocity=100 -> lower=-1.57 upper=1.57 effort=43 velocity=13.3

File: ldr-harambe-v0.3-procesed/robot_harambe_v03_fixed_axes_limits_simplified.urdf (robot description, URDF)
Before this commit: robot robot_harambe_v0.3, 26 links, 25 joints
Joints:
- joint left_ankle_pitch_joint: limit lower=-0.79 upper=0.79 effort=100 velocity=100 -> lower=-0.79 upper=0.79 effort=43 velocity=13.3
- joint left_ankle_roll_joint: limit lower=-0.79 upper=0.79 effort=100 velocity=100 -> lower=-0.79 upper=0.79 effort=43 velocity=13.3
- joint left_elbow_pitch_joint_X6: limit lower=-1.31 upper=1.83 effort=100 velocity=100 -> lower=-1.31 upper=1.83 effort=20 velocity=16.02
- joint left_hip_pitch_joint: limit lower=-2.53 upper=1.57 effort=100 velocity=100 -> lower=-2.53 upper=1.57 effort=43 velocity=13.3
- joint left_hip_roll_joint: limit lower=-0.35 upper=3.14 effort=100 velocity=100 -> lower=-0.35 upper=3.14 effort=43 velocity=13.3
- joint left_hip_yaw_joint: limit lower=-1.57 upper=1.57 effort=100 velocity=100 -> lower=-1.57 upper=1.57 effort=43 velocity=13.3
- joint left_knee_joint: limit lower=-0.17 upper=1.57 effort=100 velocity=100 -> lower=-0.17 upper=1.57 effort=43 velocity=13.3
- joint left_shoulder_pitch_joint_X6: limit lower=-3.02 upper=1.69 effort=100 velocity=100 -> lower=-3.02 upper=1.69 effort=20 velocity=16.02
- joint left_shoulder_roll_joint_X6: limit lower=-0.21 upper=2.93 effort=100 velocity=100 -> lower=-0.21 upper=2.93 effort=20 velocity=16.02
- joint left_shoulder_yaw_joint_X4: limit lower=-1.75 upper=2.97 effort=100 velocity=100 -> lower=-1.75 upper=2.97 effort=10.5 velocity=8.69
- joint left_wrist_roll_joint_X4: limit lower=-1.57 upper=1.57 effort=100 velocity=100 -> lower=-1.57 upper=1.57 effort=10.5 velocity=8.69
- joint left_wrist_yaw_joint_X4: limit lower=-2.36 upper=2.36 effort=100 velocity=100 -> lower=-2.36 upper=2.36 effort=10.5 velocity=8.69
- joint right_ankle_pitch_joint: limit lower=-0.79 upper=0.79 effort=100 velocity=100 -> lower=-0.79 upper=0.79 effort=43 velocity=13.3
- joint right_ankle_roll_joint: limit lower=-0.79 upper=0.79 effort=100 velocity=100 -> lower=-0.79 upper=0.79 effort=43 velocity=13.3
- joint right_elbow_pitch_joint_X6: limit lower=-1.31 upper=1.83 effort=100 velocity=100 -> lower=-1.31 upper=1.83 effort=20 velocity=16.02
- joint right_hip_pitch_joint: limit lower=-2.53 upper=1.57 effort=100 velocity=100 -> lower=-2.53 upper=1.57 effort=43 velocity=13.3
- joint right_hip_roll_joint: limit lower=-3.14 upper=0.35 effort=100 velocity=100 -> lower=-3.14 upper=0.35 effort=43 velocity=13.3
- joint right_hip_yaw_joint: limit lower=-1.57 upper=1.57 effort=100 velocity=100 -> lower=-1.57 upper=1.57 effort=43 velocity=13.3
- joint right_knee_joint: limit lower=-0.17 upper=1.57 effort=100 velocity=100 -> lower=-0.17 upper=1.57 effort=43 velocity=13.3
- joint right_shoulder_pitch_joint_X6: limit lower=-3.02 upper=1.69 effort=100 velocity=100 -> lower=-3.02 upper=1.69 effort=20 velocity=16.02
- joint right_shoulder_roll_joint_X6: limit lower=-2.93 upper=0.21 effort=100 velocity=100 -> lower=-2.93 upper=0.21 effort=20 velocity=16.02
- joint right_shoulder_yaw_joint_X4: limit lower=-2.97 upper=1.75 effort=100 velocity=100 -> lower=-2.97 upper=1.75 effort=10.5 velocity=8.69
- joint right_wrist_roll_joint_X4: limit lower=-1.57 upper=1.57 effort=100 velocity=100 -> lower=-1.57 upper=1.57 effort=10.5 velocity=8.69
- joint right_wrist_yaw_joint_X4: limit lower=-2.36 upper=2.36 effort=100 velocity=100 -> lower=-2.36 upper=2.36 effort=10.5 velocity=8.69
- joint waist_yaw_joint: limit lower=-1.57 upper=1.57 effort=100 velocity=100 -> lower=-1.57 upper=1.57 effort=43 velocity=13.3

File: ldr-harambe-v0.3-procesed/robot_harambe_v03_fixed_axes_limits_simplified_no_collision.urdf (robot description, URDF)
Before this commit: robot robot_harambe_v0.3, 26 links, 25 joints
Joints:
- joint left_ankle_pitch_joint: limit lower=-0.79 upper=0.79 effort=100 velocity=100 -> lower=-0.79 upper=0.79 effort=43 velocity=13.3
- joint left_ankle_roll_joint: limit lower=-0.79 upper=0.79 effort=100 velocity=100 -> lower=-0.79 upper=0.79 effort=43 velocity=13.3
- joint left_elbow_pitch_joint_X6: limit lower=-1.31 upper=1.83 effort=100 velocity=100 -> lower=-1.31 upper=1.83 effort=20 velocity=16.02
- joint left_hip_pitch_joint: limit lower=-2.53 upper=1.57 effort=100 velocity=100 -> lower=-2.53 upper=1.57 effort=43 velocity=13.3
- joint left_hip_roll_joint: limit lower=-0.35 upper=3.14 effort=100 velocity=100 -> lower=-0.35 upper=3.14 effort=43 velocity=13.3
- joint left_hip_yaw_joint: limit lower=-1.57 upper=1.57 effort=100 velocity=100 -> lower=-1.57 upper=1.57 effort=43 velocity=13.3
- joint left_knee_joint: limit lower=-0.17 upper=1.57 effort=100 velocity=100 -> lower=-0.17 upper=1.57 effort=43 velocity=13.3
- joint left_shoulder_pitch_joint_X6: limit lower=-3.02 upper=1.69 effort=100 velocity=100 -> lower=-3.02 upper=1.69 effort=20 velocity=16.02
- joint left_shoulder_roll_joint_X6: limit lower=-0.21 upper=2.93 effort=100 velocity=100 -> lower=-0.21 upper=2.93 effort=20 velocity=16.02
- joint left_shoulder_yaw_joint_X4: limit lower=-1.75 upper=2.97 effort=100 velocity=100 -> lower=-1.75 upper=2.97 effort=10.5 velocity=8.69
- joint left_wrist_roll_joint_X4: limit lower=-1.57 upper=1.57 effort=100 velocity=100 -> lower=-1.57 upper=1.57 effort=10.5 velocity=8.69
- joint left_wrist_yaw_joint_X4: limit lower=-2.36 upper=2.36 effort=100 velocity=100 -> lower=-2.36 upper=2.36 effort=10.5 velocity=8.69
- joint right_ankle_pitch_joint: limit lower=-0.79 upper=0.79 effort=100 velocity=100 -> lower=-0.79 upper=0.79 effort=43 velocity=13.3
- joint right_ankle_roll_joint: limit lower=-0.79 upper=0.79 effort=100 velocity=100 -> lower=-0.79 upper=0.79 effort=43 velocity=13.3
- joint right_elbow_pitch_joint_X6: limit lower=-1.31 upper=1.83 effort=100 velocity=100 -> lower=-1.31 upper=1.83 effort=20 velocity=16.02
- joint right_hip_pitch_joint: limit lower=-2.53 upper=1.57 effort=100 velocity=100 -> lower=-2.53 upper=1.57 effort=43 velocity=13.3
- joint right_hip_roll_joint: limit lower=-3.14 upper=0.35 effort=100 velocity=100 -> lower=-3.14 upper=0.35 effort=43 velocity=13.3
- joint right_hip_yaw_joint: limit lower=-1.57 upper=1.57 effort=100 velocity=100 -> lower=-1.57 upper=1.57 effort=43 velocity=13.3
- joint right_knee_joint: limit lower=-0.17 upper=1.57 effort=100 velocity=100 -> lower=-0.17 upper=1.57 effort=43 velocity=13.3
- joint right_shoulder_pitch_joint_X6: limit lower=-3.02 upper=1.69 effort=100 velocity=100 -> lower=-3.02 upper=1.69 effort=20 velocity=16.02
- joint right_shoulder_roll_joint_X6: limit lower=-2.93 upper=0.21 effort=100 velocity=100 -> lower=-2.93 upper=0.21 effort=20 velocity=16.02
- joint right_shoulder_yaw_joint_X4: limit lower=-2.97 upper=1.75 effort=100 velocity=100 -> lower=-2.97 upper=1.75 effort=10.5 velocity=8.69
- joint right_wrist_roll_joint_X4: limit lower=-1.57 upper=1.57 effort=100 velocity=100 -> lower=-1.57 upper=1.57 effort=10.5 velocity=8.69
- joint right_wrist_yaw_joint_X4: limit lower=-2.36 upper=2.36 effort=100 velocity=100 -> lower=-2.36 upper=2.36 effort=10.5 velocity=8.69
- joint waist_yaw_joint: limit lower=-1.57 upper=1.57 effort=100 velocity=100 -> lower=-1.57 upper=1.57 effort=43 velocity=13.3
