Commit message: udrf to urdf typo corection

File: ldr-harambe-v0.3-procesed/robot_harambe_v03.urdf (robot description, URDF)
Before this commit: robot robot_harambe_v0.3, 26 links, 25 joints
Links:
- removed link udrf_ankle_assembly
- removed link udrf_ankle_assembly_2
- added link urdf_ankle_assembly, mass 0.0818219; collision mesh filename=package://assets/urdf_ankle_assembly.stl; visual mesh filename=package://assets/urdf_ankle_assembly.stl
- added link urdf_ankle_assembly_2, mass 0.0818219; collision mesh filename=package://assets/urdf_ankle_assembly.stl; visual mesh filename=package://assets/urdf_ankle_assembly.stl
Joints:
- joint left_ankle_pitch_joint: child udrf_ankle_assembly -> urdf_ankle_assembly
- joint left_ankle_roll_joint: parent udrf_ankle_assembly -> urdf_ankle_assembly
- joint right_ankle_pitch_joint: parent udrf_ankle_assembly_2 -> urdf_ankle_assembly_2
- joint right_ankle_roll_joint: child udrf_ankle_assembly_2 -> urdf_ankle_assembly_2

File: ldr-harambe-v0.3-procesed/robot_harambe_v03_fixed_axes.urdf (robot description, URDF)
Before this commit: robot robot_harambe_v0.3, 26 links, 25 joints
Links:
- removed link udrf_ankle_assembly
- removed link udrf_ankle_assembly_2
- added link urdf_ankle_assembly, mass 0.0818219; collision mesh filename=package://assets/urdf_ankle_assembly.stl; visual mesh filename=package://assets/urdf_ankle_assembly.stl
- added link urdf_ankle_assembly_2, mass 0.0818219; collision mesh filename=package://assets/urdf_ankle_assembly.stl; visual mesh filename=package://assets/urdf_ankle_assembly.stl
Joints:
- joint left_ankle_pitch_joint: child udrf_ankle_assembly -> urdf_ankle_assembly
- joint left_ankle_roll_joint: parent udrf_ankle_assembly -> urdf_ankle_assembly
- joint right_ankle_pitch_joint: parent udrf_ankle_assembly_2 -> urdf_ankle_assembly_2
- joint right_ankle_roll_joint: child udrf_ankle_assembly_2 -> urdf_ankle_assembly_2

File: ldr-harambe-v0.3-procesed/robot_harambe_v03_fixed_axes_limits.urdf (robot description, URDF)
Before this commit: robot robot_harambe_v0.3, 26 links, 25 joints
Links:
- removed link udrf_ankle_assembly
- removed link udrf_ankle_assembly_2
- added link urdf_ankle_assembly, mass 0.0818219; collision mesh filename=package://assets/urdf_ankle_assembly.stl; visual mesh filename=package://assets/urdf_ankle_assembly.stl
- added link urdf_ankle_assembly_2, mass 0.0818219; collision mesh filename=package://assets/urdf_ankle_assembly.stl; visual mesh filename=package://assets/urdf_ankle_assembly.stl
Joints:
- joint left_ankle_pitch_joint: child udrf_ankle_assembly -> urdf_ankle_assembly
- joint left_ankle_roll_joint: parent udrf_ankle_assembly -> urdf_ankle_assembly
- joint right_ankle_pitch_joint: parent udrf_ankle_assembly_2 -> urdf_ankle_assembly_2
- joint right_ankle_roll_joint: child udrf_ankle_assembly_2 -> urdf_ankle_assembly_2

File: ldr-harambe-v0.3-procesed/robot_harambe_v03_fixed_axes_limits_simplified.urdf (robot description, URDF)
Before this commit: robot robot_harambe_v0.3, 26 links, 25 joints
Links:
- removed link udrf_ankle_assembly
- removed link udrf_ankle_assembly_2
- added link urdf_ankle_assembly, mass 0.0818219; collision mesh filename=package://meshes/collision/urdf_ankle_assembly.stl; visual mesh filename=package://meshes/visual/urdf_ankle_assembly.stl
- added link urdf_ankle_assembly_2, mass 0.0818219; collision mesh filename=package://meshes/collision/urdf_ankle_assembly.stl; visual mesh filename=package://meshes/visual/urdf_ankle_assembly.stl
Joints:
- joint left_ankle_pitch_joint: child udrf_ankle_assembly -> urdf_ankle_assembly
- joint left_ankle_roll_joint: parent udrf_ankle_assembly -> urdf_ankle_assembly
- joint right_ankle_pitch_joint: parent udrf_ankle_assembly_2 -> urdf_ankle_assembly_2
- joint right_ankle_roll_joint: child udrf_ankle_assembly_2 -> urdf_ankle_assembly_2

Commit message: update joints name and limits

File: ldr-harambe-v0.3-procesed/robot_harambe_v03.urdf (robot description, URDF)
Before this commit: robot robot_harambe_v0.3, 26 links, 25 joints
Joints:
- removed joint left_ankle_pitch_joint
- removed joint left_ankle_roll_joint
- removed joint left_hip_pitch_joint
- removed joint left_hip_roll_joint
- removed joint left_hip_yaw_joint
- removed joint left_knee_joint
- removed joint right_ankle_pitch_joint
- removed joint right_ankle_roll_joint
- removed joint right_hip_pitch_joint
- removed joint right_hip_roll_joint
- removed joint right_hip_yaw_joint
- removed joint right_knee_joint
- removed joint waist_yaw_joint
- added joint left_ankle_pitch_joint_X4: type revolute, parent urdf_l_tibia_assembly, child urdf_ankle_assembly, origin xyz=0 0.395 -0.051 rpy=0 -0 0, axis 0 0 1, limit lower=-0.785398 upper=0.785398 effort=10 velocity=10
- added joint left_ankle_roll_joint_X4: type revolute, parent urdf_ankle_assembly, child urdf_foot_assembly, origin xyz=-0.012 0.028 -0.004 rpy=0 1.5708 0, axis 0 0 1, limit lower=-0.785398 upper=0.785398 effort=10 velocity=10
- added joint left_hip_pitch_joint_X8: type revolute, parent urdf_base, child urdf_hip_assembly, origin xyz=-0.111301 0.0333787 -0.467748 rpy=-1.5708 -0 1.5708, axis 0 0 1, limit lower=-2.53073 upper=1.5708 effort=10 velocity=10
- added joint left_hip_roll_joint_X8: type revolute, parent urdf_hip_assembly, child urdf_l_upper_femur_assembly, origin xyz=0.055 0 0.073 rpy=-0 1.5708 0, axis 0 0 1, limit lower=-0.349066 upper=3.14159 effort=10 velocity=10
- added joint left_hip_yaw_joint_X8: type revolute, parent urdf_l_upper_femur_assembly, child urdf_lower_femur_assembly, origin xyz=-0 0.217 -0.053 rpy=-1.5708 0 0, axis 0 0 1, limit lower=-1.5708 upper=1.5708 effort=10 velocity=10
- added joint left_knee_joint_X8: type revolute, parent urdf_lower_femur_assembly, child urdf_l_tibia_assembly, origin xyz=-0.055 0 0.113 rpy=1.5708 0 -1.5708, axis 0 0 1, limit lower=-0.174533 upper=1.5708 effort=10 velocity=10
- added joint right_ankle_pitch_joint_X4: type revolute, parent urdf_ankle_assembly_2, child urdf_foot_assembly_2, origin xyz=-0.012 0.028 -0.004 rpy=0 1.5708 0, axis 0 0 1, limit lower=-0.785398 upper=0.785398 effort=10 velocity=10
- added joint right_ankle_roll_joint_X4: type revolute, parent urdf_r_tibia_assembly, child urdf_ankle_assembly_2, origin xyz=-0 0.395 0.059 rpy=0 -0 0, axis 0 0 1, limit lower=-0.785398 upper=0.785398 effort=10 velocity=10
- added joint right_hip_pitch_joint_X8: type revolute, parent urdf_base, child urdf_hip_assembly_2, origin xyz=0.107699 0.0333787 -0.467748 rpy=1.5708 -0 1.5708, axis 0 0 1, limit lower=-1.5708 upper=2.53073 effort=10 velocity=10
- added joint right_hip_roll_joint_X8: type revolute, parent urdf_hip_assembly_2, child urdf_r_upper_femur_assemby, origin xyz=0.055 0 0.078 rpy=-3.14159 -1.5708 0, axis 0 0 1, limit lower=-3.14159 upper=0.349066 effort=10 velocity=10
- added joint right_hip_yaw_joint_X8: type revolute, parent urdf_r_upper_femur_assemby, child urdf_lower_femur_assembly_2, origin xyz=0 0.217 -0.053 rpy=-1.5708 0 -0, axis 0 0 1, limit lower=-1.5708 upper=1.5708 effort=10 velocity=10
- added joint right_knee_joint_X8: type revolute, parent urdf_lower_femur_assembly_2, child urdf_r_tibia_assembly, origin xyz=0.055 -0 0.113 rpy=1.5708 0 -1.5708, axis 0 0 1, limit lower=-0.174533 upper=1.5708 effort=10 velocity=10
- added joint waist_yaw_joint_X8: type revolute, parent urdf_base, child urdf_simplified_torso, origin xyz=0.000698852 0.0333787 -0.300748 rpy=0 -0 0, axis 0 0 1, limit lower=-1.5708 upper=1.5708 effort=10 velocity=10

File: ldr-harambe-v0.3-procesed/robot_harambe_v03_fixed_axes.urdf (robot description, URDF)
Before this commit: robot robot_harambe_v0.3, 26 links, 25 joints
Joints:
- removed joint left_ankle_pitch_joint
- removed joint left_ankle_roll_joint
- removed joint left_hip_pitch_joint
- removed joint left_hip_roll_joint
- removed joint left_hip_yaw_joint
- removed joint left_knee_joint
- removed joint right_ankle_pitch_joint
- removed joint right_ankle_roll_joint
- removed joint right_hip_pitch_joint
- removed joint right_hip_roll_joint
- removed joint right_hip_yaw_joint
- removed joint right_knee_joint
- removed joint waist_yaw_joint
- added joint left_ankle_pitch_joint_X4: type revolute, parent urdf_l_tibia_assembly, child urdf_ankle_assembly, origin xyz=-1.45092e-06 -0.051 -0.395 rpy=0 0 0, axis 0 1 0, limit lower=-0.785398 upper=0.785398 effort=10 velocity=10
- added joint left_ankle_roll_joint_X4: type revolute, parent urdf_ankle_assembly, child urdf_foot_assembly, origin xyz=-0.0120001 -0.004 -0.028 rpy=0 0 0, axis 1 0 0, limit lower=-0.785398 upper=0.785398 effort=10 velocity=10
- added joint left_hip_pitch_joint_X8: type revolute, parent urdf_base, child urdf_hip_assembly, origin xyz=0.0333787 0.111301 -0.467748 rpy=0 0 0, axis 0 1 0, limit lower=-2.53073 upper=1.5708 effort=10 velocity=10
- added joint left_hip_roll_joint_X8: type revolute, parent urdf_hip_assembly, child urdf_l_upper_femur_assembly, origin xyz=0.055 0.073 0 rpy=0 0 0, axis 1 0 0, limit lower=-0.349066 upper=3.14159 effort=10 velocity=10
- added joint left_hip_yaw_joint_X8: type revolute, parent urdf_l_upper_femur_assembly, child urdf_lower_femur_assembly, origin xyz=-0.053 -7.97086e-07 -0.217 rpy=0 0 0, axis 0 0 1, limit lower=-1.5708 upper=1.5708 effort=10 velocity=10
- added joint left_knee_joint_X8: type revolute, parent urdf_lower_femur_assembly, child urdf_l_tibia_assembly, origin xyz=0 0.055 -0.113 rpy=0 0 0, axis 0 1 0, limit lower=-0.174533 upper=1.5708 effort=10 velocity=10
- added joint right_ankle_pitch_joint_X4: type revolute, parent urdf_ankle_assembly_2, child urdf_foot_assembly_2, origin xyz=-0.012 -0.004 -0.028 rpy=0 0 0, axis 1 0 0, limit lower=-0.785398 upper=0.785398 effort=10 velocity=10
- added joint right_ankle_roll_joint_X4: type revolute, parent urdf_r_tibia_assembly, child urdf_ankle_assembly_2, origin xyz=-4.02748e-07 0.059 -0.395 rpy=0 0 0, axis 0 1 0, limit lower=-0.785398 upper=0.785398 effort=10 velocity=10
- added joint right_hip_pitch_joint_X8: type revolute, parent urdf_base, child urdf_hip_assembly_2, origin xyz=0.0333787 -0.107699 -0.467748 rpy=0 0 0, axis 0 1 0, limit lower=-2.53073 upper=1.5708 effort=10 velocity=10
- added joint right_hip_roll_joint_X8: type revolute, parent urdf_hip_assembly_2, child urdf_r_upper_femur_assemby, origin xyz=0.055 -0.078 0 rpy=0 0 0, axis 1 0 0, limit lower=-3.14159 upper=0.349066 effort=10 velocity=10
- added joint right_hip_yaw_joint_X8: type revolute, parent urdf_r_upper_femur_assemby, child urdf_lower_femur_assembly_2, origin xyz=-0.053 7.97086e-07 -0.217 rpy=0 0 0, axis 0 0 1, limit lower=-1.5708 upper=1.5708 effort=10 velocity=10
- added joint right_knee_joint_X8: type revolute, parent urdf_lower_femur_assembly_2, child urdf_r_tibia_assembly, origin xyz=0 -0.055 -0.113 rpy=0 0 0, axis 0 1 0, limit lower=-0.174533 upper=1.5708 effort=10 velocity=10
- added joint waist_yaw_joint_X8: type revolute, parent urdf_base, child urdf_simplified_torso, origin xyz=0.0333787 -0.000698852 -0.300748 rpy=0 0 0, axis 0 0 1, limit lower=-1.5708 upper=1.5708 effort=10 velocity=10

File: ldr-harambe-v0.3-procesed/robot_harambe_v03_fixed_axes_limits.urdf (robot description, URDF)
Before this commit: robot robot_harambe_v0.3, 26 links, 25 joints
Joints:
- removed joint left_ankle_pitch_joint
- removed joint left_ankle_roll_joint
- removed joint left_hip_pitch_joint
- removed joint left_hip_roll_joint
- removed joint left_hip_yaw_joint
- removed joint left_knee_joint
- removed joint right_ankle_pitch_joint
- removed joint right_ankle_roll_joint
- removed joint right_hip_pitch_joint
- removed joint right_hip_roll_joint
- removed joint right_hip_yaw_joint
- removed joint right_knee_joint
- removed joint waist_yaw_joint
- added joint left_ankle_pitch_joint_X4: type revolute, parent urdf_l_tibia_assembly, child urdf_ankle_assembly, origin xyz=-1.45092e-06 -0.051 -0.395 rpy=0 0 0, axis 0 1 0, limit lower=-0.79 upper=0.79 effort=10.5 velocity=8.69
- added joint left_ankle_roll_joint_X4: type revolute, parent urdf_ankle_assembly, child urdf_foot_assembly, origin xyz=-0.0120001 -0.004 -0.028 rpy=0 0 0, axis 1 0 0, limit lower=-0.79 upper=0.79 effort=10.5 velocity=8.69
- added joint left_hip_pitch_joint_X8: type revolute, parent urdf_base, child urdf_hip_assembly, origin xyz=0.0333787 0.111301 -0.467748 rpy=0 0 0, axis 0 1 0, limit lower=-2.53 upper=1.57 effort=43 velocity=13.3
- added joint left_hip_roll_joint_X8: type revolute, parent urdf_hip_assembly, child urdf_l_upper_femur_assembly, origin xyz=0.055 0.073 0 rpy=0 0 0, axis 1 0 0, limit lower=-0.35 upper=3.14 effort=43 velocity=13.3
- added joint left_hip_yaw_joint_X8: type revolute, parent urdf_l_upper_femur_assembly, child urdf_lower_femur_assembly, origin xyz=-0.053 -7.97086e-07 -0.217 rpy=0 0 0, axis 0 0 1, limit lower=-1.57 upper=1.57 effort=43 velocity=13.3
- added joint left_knee_joint_X8: type revolute, parent urdf_lower_femur_assembly, child urdf_l_tibia_assembly, origin xyz=0 0.055 -0.113 rpy=0 0 0, axis 0 1 0, limit lower=-0.17 upper=1.57 effort=43 velocity=13.3
- added joint right_ankle_pitch_joint_X4: type revolute, parent urdf_ankle_assembly_2, child urdf_foot_assembly_2, origin xyz=-0.012 -0.004 -0.028 rpy=0 0 0, axis 1 0 0, limit lower=-0.79 upper=0.79 effort=10.5 velocity=8.69
- added joint right_ankle_roll_joint_X4: type revolute, parent urdf_r_tibia_assembly, child urdf_ankle_assembly_2, origin xyz=-4.02748e-07 0.059 -0.395 rpy=0 0 0, axis 0 1 0, limit lower=-0.79 upper=0.79 effort=10.5 velocity=8.69
- added joint right_hip_pitch_joint_X8: type revolute, parent urdf_base, child urdf_hip_assembly_2, origin xyz=0.0333787 -0.107699 -0.467748 rpy=0 0 0, axis 0 1 0, limit lower=-2.53 upper=1.57 effort=43 velocity=13.3
- added joint right_hip_roll_joint_X8: type revolute, parent urdf_hip_assembly_2, child urdf_r_upper_femur_assemby, origin xyz=0.055 -0.078 0 rpy=0 0 0, axis 1 0 0, limit lower=-3.14 upper=0.35 effort=43 velocity=13.3
- added joint right_hip_yaw_joint_X8: type revolute, parent urdf_r_upper_femur_assemby, child urdf_lower_femur_assembly_2, origin xyz=-0.053 7.97086e-07 -0.217 rpy=0 0 0, axis 0 0 1, limit lower=-1.57 upper=1.57 effort=43 velocity=13.3
- added joint right_knee_joint_X8: type revolute, parent urdf_lower_femur_assembly_2, child urdf_r_tibia_assembly, origin xyz=0 -0.055 -0.113 rpy=0 0 0, axis 0 1 0, limit lower=-0.17 upper=1.57 effort=43 velocity=13.3
- added joint waist_yaw_joint_X8: type revolute, parent urdf_base, child urdf_simplified_torso, origin xyz=0.0333787 -0.000698852 -0.300748 rpy=0 0 0, axis 0 0 1, limit lower=-1.57 upper=1.57 effort=43 velocity=13.3

File: ldr-harambe-v0.3-procesed/robot_harambe_v03_fixed_axes_limits_simplified.urdf (robot description, URDF)
Before this commit: robot robot_harambe_v0.3, 26 links, 25 joints
Joints:
- removed joint left_ankle_pitch_joint
- removed joint left_ankle_roll_joint
- removed joint left_hip_pitch_joint
- removed joint left_hip_roll_joint
- removed joint left_hip_yaw_joint
- removed joint left_knee_joint
- removed joint right_ankle_pitch_joint
- removed joint right_ankle_roll_joint
- removed joint right_hip_pitch_joint
- removed joint right_hip_roll_joint
- removed joint right_hip_yaw_joint
- removed joint right_knee_joint
- removed joint waist_yaw_joint
- added joint left_ankle_pitch_joint_X4: type revolute, parent urdf_l_tibia_assembly, child urdf_ankle_assembly, origin xyz=-1.45092e-06 -0.051 -0.395 rpy=0 0 0, axis 0 1 0, limit lower=-0.79 upper=0.79 effort=10.5 velocity=8.69
- added joint left_ankle_roll_joint_X4: type revolute, parent urdf_ankle_assembly, child urdf_foot_assembly, origin xyz=-0.0120001 -0.004 -0.028 rpy=0 0 0, axis 1 0 0, limit lower=-0.79 upper=0.79 effort=10.5 velocity=8.69
- added joint left_hip_pitch_joint_X8: type revolute, parent urdf_base, child urdf_hip_assembly, origin xyz=0.0333787 0.111301 -0.467748 rpy=0 0 0, axis 0 1 0, limit lower=-2.53 upper=1.57 effort=43 velocity=13.3
- added joint left_hip_roll_joint_X8: type revolute, parent urdf_hip_assembly, child urdf_l_upper_femur_assembly, origin xyz=0.055 0.073 0 rpy=0 0 0, axis 1 0 0, limit lower=-0.35 upper=3.14 effort=43 velocity=13.3
- added joint left_hip_yaw_joint_X8: type revolute, parent urdf_l_upper_femur_assembly, child urdf_lower_femur_assembly, origin xyz=-0.053 -7.97086e-07 -0.217 rpy=0 0 0, axis 0 0 1, limit lower=-1.57 upper=1.57 effort=43 velocity=13.3
- added joint left_knee_joint_X8: type revolute, parent urdf_lower_femur_assembly, child urdf_l_tibia_assembly, origin xyz=0 0.055 -0.113 rpy=0 0 0, axis 0 1 0, limit lower=-0.17 upper=1.57 effort=43 velocity=13.3
- added joint right_ankle_pitch_joint_X4: type revolute, parent urdf_ankle_assembly_2, child urdf_foot_assembly_2, origin xyz=-0.012 -0.004 -0.028 rpy=0 0 0, axis 1 0 0, limit lower=-0.79 upper=0.79 effort=10.5 velocity=8.69
- added joint right_ankle_roll_joint_X4: type revolute, parent urdf_r_tibia_assembly, child urdf_ankle_assembly_2, origin xyz=-4.02748e-07 0.059 -0.395 rpy=0 0 0, axis 0 1 0, limit lower=-0.79 upper=0.79 effort=10.5 velocity=8.69
- added joint right_hip_pitch_joint_X8: type revolute, parent urdf_base, child urdf_hip_assembly_2, origin xyz=0.0333787 -0.107699 -0.467748 rpy=0 0 0, axis 0 1 0, limit lower=-2.53 upper=1.57 effort=43 velocity=13.3
- added joint right_hip_roll_joint_X8: type revolute, parent urdf_hip_assembly_2, child urdf_r_upper_femur_assemby, origin xyz=0.055 -0.078 0 rpy=0 0 0, axis 1 0 0, limit lower=-3.14 upper=0.35 effort=43 velocity=13.3
- added joint right_hip_yaw_joint_X8: type revolute, parent urdf_r_upper_femur_assemby, child urdf_lower_femur_assembly_2, origin xyz=-0.053 7.97086e-07 -0.217 rpy=0 0 0, axis 0 0 1, limit lower=-1.57 upper=1.57 effort=43 velocity=13.3
- added joint right_knee_joint_X8: type revolute, parent urdf_lower_femur_assembly_2, child urdf_r_tibia_assembly, origin xyz=0 -0.055 -0.113 rpy=0 0 0, axis 0 1 0, limit lower=-0.17 upper=1.57 effort=43 velocity=13.3
- added joint waist_yaw_joint_X8: type revolute, parent urdf_base, child urdf_simplified_torso, origin xyz=0.0333787 -0.000698852 -0.300748 rpy=0 0 0, axis 0 0 1, limit lower=-1.57 upper=1.57 effort=43 velocity=13.3
