Commit message: don t use aply limits

File: ldr-harambe-v0.4/robot_harambe_v04_fixed_axes_simplified.urdf (robot description, URDF)
Before this commit: robot robot_harambe_v04, 26 links, 25 joints
Joints:
- joint left_ankle_pitch_joint_X4: limit lower=-0.79 upper=0.79 effort=10.5 velocity=8.69 -> lower=-0.785398 upper=0.785398 effort=10 velocity=10
- joint left_ankle_roll_joint_X4: limit lower=-0.79 upper=0.79 effort=10.5 velocity=8.69 -> lower=-0.785398 upper=0.785398 effort=10 velocity=10
- joint left_elbow_pitch_joint_X6: limit lower=-1.31 upper=1.83 effort=20 velocity=16.02 -> lower=-1.309 upper=1.8326 effort=10 velocity=10
- joint left_hip_pitch_joint_X8: limit lower=-2.53 upper=1.57 effort=43 velocity=13.3 -> lower=-2.61799 upper=2.61799 effort=10 velocity=10
- joint left_hip_roll_joint_X8: limit lower=-0.35 upper=3.14 effort=43 velocity=13.3 -> lower=-0.383972 upper=3.22886 effort=10 velocity=10
- joint left_hip_yaw_joint_X8: limit lower=-1.57 upper=1.57 effort=43 velocity=13.3 -> lower=-2.15199 upper=2.09003 effort=10 velocity=10
- joint left_knee_joint_X8: limit lower=-0.17 upper=1.57 effort=43 velocity=13.3 -> lower=-1.52716 upper=1.52716 effort=10 velocity=10
- joint left_shoulder_pitch_joint_X6: limit lower=-3.02 upper=1.69 effort=20 velocity=16.02 -> lower=-3.01942 upper=1.69297 effort=10 velocity=10
- joint left_shoulder_roll_joint_X6: limit lower=-0.21 upper=2.93 effort=20 velocity=16.02 -> lower=-0.20944 upper=2.93215 effort=10 velocity=10
- joint left_shoulder_yaw_joint_X4: limit lower=-1.75 upper=2.97 effort=10.5 velocity=8.69 -> lower=-1.74533 upper=2.96706 effort=10 velocity=10
- joint left_wrist_roll_joint_X4: limit lower=-1.57 upper=1.57 effort=10.5 velocity=8.69 -> lower=-1.5708 upper=1.5708 effort=10 velocity=10
- joint left_wrist_yaw_joint_X4: limit lower=-2.36 upper=2.36 effort=10.5 velocity=8.69 -> lower=-2.35619 upper=2.35619 effort=10 velocity=10
- joint right_ankle_pitch_joint_X4: limit lower=-0.79 upper=0.79 effort=10.5 velocity=8.69 -> lower=-0.785398 upper=0.785398 effort=10 velocity=10
- joint right_ankle_roll_joint_X4: limit lower=-0.79 upper=0.79 effort=10.5 velocity=8.69 -> lower=-0.785398 upper=0.785398 effort=10 velocity=10
- joint right_elbow_pitch_joint_X6: limit lower=-1.31 upper=1.83 effort=20 velocity=16.02 -> lower=-1.309 upper=1.8326 effort=10 velocity=10
- joint right_hip_pitch_joint_X8: limit lower=-2.53 upper=1.57 effort=43 velocity=13.3 -> lower=-2.61799 upper=2.61799 effort=10 velocity=10
- joint right_hip_roll_joint_X8: limit lower=-3.14 upper=0.35 effort=43 velocity=13.3 -> lower=-3.22886 upper=0.383972 effort=10 velocity=10
- joint right_hip_yaw_joint_X8: limit lower=-1.57 upper=1.57 effort=43 velocity=13.3 -> lower=-1.5708 upper=1.5708 effort=10 velocity=10
- joint right_knee_joint_X8: limit lower=-0.17 upper=1.57 effort=43 velocity=13.3 -> lower=-1.52716 upper=1.52716 effort=10 velocity=10
- joint right_shoulder_pitch_joint_X6: limit lower=-3.02 upper=1.69 effort=20 velocity=16.02 -> lower=-3.01942 upper=1.69297 effort=10 velocity=10
- joint right_shoulder_roll_joint_X6: limit lower=-2.93 upper=0.21 effort=20 velocity=16.02 -> lower=-2.93215 upper=0.20944 effort=10 velocity=10
- joint right_shoulder_yaw_joint_X4: limit lower=-2.97 upper=1.75 effort=10.5 velocity=8.69 -> lower=-2.96706 upper=1.74533 effort=10 velocity=10
- joint right_wrist_roll_joint_X4: limit lower=-1.57 upper=1.57 effort=10.5 velocity=8.69 -> lower=-1.65806 upper=1.65806 effort=10 velocity=10
- joint right_wrist_yaw_joint_X4: limit lower=-2.36 upper=2.36 effort=10.5 velocity=8.69 -> lower=-2.35619 upper=2.35619 effort=10 velocity=10
- joint waist_yaw_joint_X8: limit lower=-1.57 upper=1.57 effort=43 velocity=13.3 -> lower=-2.60054 upper=2.60054 effort=10 velocity=10

File: ldr-harambe-v0.4/robot_harambe_v04_fixed_axes_simplified_no_collision.urdf (robot description, URDF)
Before this commit: robot robot_harambe_v04, 26 links, 25 joints
Joints:
- joint left_ankle_pitch_joint_X4: limit lower=-0.79 upper=0.79 effort=10.5 velocity=8.69 -> lower=-0.785398 upper=0.785398 effort=10 velocity=10
- joint left_ankle_roll_joint_X4: limit lower=-0.79 upper=0.79 effort=10.5 velocity=8.69 -> lower=-0.785398 upper=0.785398 effort=10 velocity=10
- joint left_elbow_pitch_joint_X6: limit lower=-1.31 upper=1.83 effort=20 velocity=16.02 -> lower=-1.309 upper=1.8326 effort=10 velocity=10
- joint left_hip_pitch_joint_X8: limit lower=-2.53 upper=1.57 effort=43 velocity=13.3 -> lower=-2.61799 upper=2.61799 effort=10 velocity=10
- joint left_hip_roll_joint_X8: limit lower=-0.35 upper=3.14 effort=43 velocity=13.3 -> lower=-0.383972 upper=3.22886 effort=10 velocity=10
- joint left_hip_yaw_joint_X8: limit lower=-1.57 upper=1.57 effort=43 velocity=13.3 -> lower=-2.15199 upper=2.09003 effort=10 velocity=10
- joint left_knee_joint_X8: limit lower=-0.17 upper=1.57 effort=43 velocity=13.3 -> lower=-1.52716 upper=1.52716 effort=10 velocity=10
- joint left_shoulder_pitch_joint_X6: limit lower=-3.02 upper=1.69 effort=20 velocity=16.02 -> lower=-3.01942 upper=1.69297 effort=10 velocity=10
- joint left_shoulder_roll_joint_X6: limit lower=-0.21 upper=2.93 effort=20 velocity=16.02 -> lower=-0.20944 upper=2.93215 effort=10 velocity=10
- joint left_shoulder_yaw_joint_X4: limit lower=-1.75 upper=2.97 effort=10.5 velocity=8.69 -> lower=-1.74533 upper=2.96706 effort=10 velocity=10
- joint left_wrist_roll_joint_X4: limit lower=-1.57 upper=1.57 effort=10.5 velocity=8.69 -> lower=-1.5708 upper=1.5708 effort=10 velocity=10
- joint left_wrist_yaw_joint_X4: limit lower=-2.36 upper=2.36 effort=10.5 velocity=8.69 -> lower=-2.35619 upper=2.35619 effort=10 velocity=10
- joint right_ankle_pitch_joint_X4: limit lower=-0.79 upper=0.79 effort=10.5 velocity=8.69 -> lower=-0.785398 upper=0.785398 effort=10 velocity=10
- joint right_ankle_roll_joint_X4: limit lower=-0.79 upper=0.79 effort=10.5 velocity=8.69 -> lower=-0.785398 upper=0.785398 effort=10 velocity=10
- joint right_elbow_pitch_joint_X6: limit lower=-1.31 upper=1.83 effort=20 velocity=16.02 -> lower=-1.309 upper=1.8326 effort=10 velocity=10
- joint right_hip_pitch_joint_X8: limit lower=-2.53 upper=1.57 effort=43 velocity=13.3 -> lower=-2.61799 upper=2.61799 effort=10 velocity=10
- joint right_hip_roll_joint_X8: limit lower=-3.14 upper=0.35 effort=43 velocity=13.3 -> lower=-3.22886 upper=0.383972 effort=10 velocity=10
- joint right_hip_yaw_joint_X8: limit lower=-1.57 upper=1.57 effort=43 velocity=13.3 -> lower=-1.5708 upper=1.5708 effort=10 velocity=10
- joint right_knee_joint_X8: limit lower=-0.17 upper=1.57 effort=43 velocity=13.3 -> lower=-1.52716 upper=1.52716 effort=10 velocity=10
- joint right_shoulder_pitch_joint_X6: limit lower=-3.02 upper=1.69 effort=20 velocity=16.02 -> lower=-3.01942 upper=1.69297 effort=10 velocity=10
- joint right_shoulder_roll_joint_X6: limit lower=-2.93 upper=0.21 effort=20 velocity=16.02 -> lower=-2.93215 upper=0.20944 effort=10 velocity=10
- joint right_shoulder_yaw_joint_X4: limit lower=-2.97 upper=1.75 effort=10.5 velocity=8.69 -> lower=-2.96706 upper=1.74533 effort=10 velocity=10
- joint right_wrist_roll_joint_X4: limit lower=-1.57 upper=1.57 effort=10.5 velocity=8.69 -> lower=-1.65806 upper=1.65806 effort=10 velocity=10
- joint right_wrist_yaw_joint_X4: limit lower=-2.36 upper=2.36 effort=10.5 velocity=8.69 -> lower=-2.35619 upper=2.35619 effort=10 velocity=10
- joint waist_yaw_joint_X8: limit lower=-1.57 upper=1.57 effort=43 velocity=13.3 -> lower=-2.60054 upper=2.60054 effort=10 velocity=10

File: ldr-harambe-v0.4/urdf/joints/body_joints.xacro (robot description, xacro)
@@ -19,6 +19,6 @@
     <child link="urdf_simplified_torso"/>
     <axis xyz="0 0 1"/>
-    <limit effort="${X8_moderate_effort}" velocity="${X8_rated_velocity}" lower="-1.57" upper="1.57"/>
-    <dynamics friction="${X8_friction}" damping="${X8_damping}"/>
+    <limit effort="${X8_moderate_effort}" velocity="${X8_rated_velocity}" lower="-2.60054" upper="2.60054"/>
+    <dynamics damping="${X8_damping}" friction="${X8_friction}"/>
   </joint>
 </robot>

File: ldr-harambe-v0.4/urdf/joints/left_arm_joints.xacro (robot description, xacro)
@@ -9,6 +9,6 @@
     <child link="urdf_l_shoulder_assembly"/>
     <axis xyz="0 1 0"/>
-    <limit effort="${X6_moderate_effort}" velocity="${X6_rated_velocity}" lower="-3.02" upper="1.69"/>
-    <dynamics friction="${X6_friction}" damping="${X6_damping}"/>
+    <limit effort="${X6_moderate_effort}" velocity="${X6_rated_velocity}" lower="-3.01942" upper="1.69297"/>
+    <dynamics damping="${X6_damping}" friction="${X6_friction}"/>
   </joint>
   <joint name="left_shoulder_roll_joint_X6" type="revolute">
@@ -17,6 +17,6 @@
     <child link="urdf_l_upper_arm_assembly"/>
     <axis xyz="1 0 0"/>
-    <limit effort="${X6_moderate_effort}" velocity="${X6_rated_velocity}" lower="-0.21" upper="2.93"/>
-    <dynamics friction="${X6_friction}" damping="${X6_damping}"/>
+    <limit effort="${X6_moderate_effort}" velocity="${X6_rated_velocity}" lower="-0.20944" upper="2.93215"/>
+    <dynamics damping="${X6_damping}" friction="${X6_friction}"/>
   </joint>
   <joint name="left_shoulder_yaw_joint_X4" type="revolute">
@@ -25,6 +25,6 @@
     <child link="urdf_l_elbow_assembly"/>
     <axis xyz="0 0 1"/>
-    <limit effort="${X4_moderate_effort}" velocity="${X4_rated_velocity}" lower="-1.75" upper="2.97"/>
-    <dynamics friction="${X4_friction}" damping="${X4_damping}"/>
+    <limit effort="${X4_moderate_effort}" velocity="${X4_rated_velocity}" lower="-1.74533" upper="2.96706"/>
+    <dynamics damping="${X4_damping}" friction="${X4_friction}"/>
   </joint>
   <joint name="left_elbow_pitch_joint_X6" type="revolute">
@@ -33,6 +33,6 @@
     <child link="urdf_l_upper_forearm_assembly"/>
     <axis xyz="0 1 0"/>
-    <limit effort="${X6_moderate_effort}" velocity="${X6_rated_velocity}" lower="-1.31" upper="1.83"/>
-    <dynamics friction="${X6_friction}" damping="${X6_damping}"/>
+    <limit effort="${X6_moderate_effort}" velocity="${X6_rated_velocity}" lower="-1.309" upper="1.8326"/>
+    <dynamics damping="${X6_damping}" friction="${X6_friction}"/>
   </joint>
   <joint name="left_wrist_yaw_joint_X4" type="revolute">
@@ -41,6 +41,6 @@
     <child link="urdf_l_lower_forearm_assembly"/>
     <axis xyz="0 0 1"/>
-    <limit effort="${X4_moderate_effort}" velocity="${X4_rated_velocity}" lower="-2.36" upper="2.36"/>
-    <dynamics friction="${X4_friction}" damping="${X4_damping}"/>
+    <limit effort="${X4_moderate_effort}" velocity="${X4_rated_velocity}" lower="-2.35619" upper="2.35619"/>
+    <dynamics damping="${X4_damping}" friction="${X4_friction}"/>
   </joint>
   <joint name="left_wrist_roll_joint_X4" type="revolute">
@@ -49,6 +49,6 @@
     <child link="urdf_l_wrist_assembly"/>
     <axis xyz="1 0 0"/>
-    <limit effort="${X4_moderate_effort}" velocity="${X4_rated_velocity}" lower="-1.57" upper="1.57"/>
-    <dynamics friction="${X4_friction}" damping="${X4_damping}"/>
+    <limit effort="${X4_moderate_effort}" velocity="${X4_rated_velocity}" lower="-1.5708" upper="1.5708"/>
+    <dynamics damping="${X4_damping}" friction="${X4_friction}"/>
   </joint>
 </robot>

File: ldr-harambe-v0.4/urdf/joints/left_foot_joints.xacro (robot description, xacro)
@@ -9,6 +9,6 @@
     <child link="urdf_hip_assembly"/>
     <axis xyz="0 1 0"/>
-    <limit effort="${X8_moderate_effort}" velocity="${X8_rated_velocity}" lower="-2.53" upper="1.57"/>
-    <dynamics friction="${X8_friction}" damping="${X8_damping}"/>
+    <limit effort="${X8_moderate_effort}" velocity="${X8_rated_velocity}" lower="-2.61799" upper="2.61799"/>
+    <dynamics damping="${X8_damping}" friction="${X8_friction}"/>
   </joint>
   <joint name="left_hip_roll_joint_X8" type="${leg_joint_type}">
@@ -17,6 +17,6 @@
     <child link="urdf_l_upper_femur_assembly"/>
     <axis xyz="1 0 0"/>
-    <limit effort="${X8_moderate_effort}" velocity="${X8_rated_velocity}" lower="-0.35" upper="3.14"/>
-    <dynamics friction="${X8_friction}" damping="${X8_damping}"/>
+    <limit effort="${X8_moderate_effort}" velocity="${X8_rated_velocity}" lower="-0.383972" upper="3.22886"/>
+    <dynamics damping="${X8_damping}" friction="${X8_friction}"/>
   </joint>
   <joint name="left_hip_yaw_joint_X8" type="${leg_joint_type}">
@@ -25,6 +25,6 @@
     <child link="urdf_lower_femur_assembly"/>
     <axis xyz="0 0 1"/>
-    <limit effort="${X8_moderate_effort}" velocity="${X8_rated_velocity}" lower="-1.57" upper="1.57"/>
-    <dynamics friction="${X8_friction}" damping="${X8_damping}"/>
+    <limit effort="${X8_moderate_effort}" velocity="${X8_rated_velocity}" lower="-2.15199" upper="2.09003"/>
+    <dynamics damping="${X8_damping}" friction="${X8_friction}"/>
   </joint>
   <joint name="left_knee_joint_X8" type="${leg_joint_type}">
@@ -33,6 +33,6 @@
     <child link="urdf_l_tibia_assembly"/>
     <axis xyz="0 1 0"/>
-    <limit effort="${X8_moderate_effort}" velocity="${X8_rated_velocity}" lower="-0.17" upper="1.57"/>
-    <dynamics friction="${X8_friction}" damping="${X8_damping}"/>
+    <limit effort="${X8_moderate_effort}" velocity="${X8_rated_velocity}" lower="-1.52716" upper="1.52716"/>
+    <dynamics damping="${X8_damping}" friction="${X8_friction}"/>
   </joint>
   <joint name="left_ankle_pitch_joint_X4" type="${leg_joint_type}">
@@ -41,6 +41,6 @@
     <child link="udrf_ankle_assembly"/>
     <axis xyz="0 1 0"/>
-    <limit effort="${X4_moderate_effort}" velocity="${X4_rated_velocity}" lower="-0.79" upper="0.79"/>
-    <dynamics friction="${X4_friction}" damping="${X4_damping}"/>
+    <limit effort="${X4_moderate_effort}" velocity="${X4_rated_velocity}" lower="-0.785398" upper="0.785398"/>
+    <dynamics damping="${X4_damping}" friction="${X4_friction}"/>
   </joint>
   <joint name="left_ankle_roll_joint_X4" type="${leg_joint_type}">
@@ -49,6 +49,6 @@
     <child link="urdf_foot_assembly"/>
     <axis xyz="1 0 0"/>
-    <limit effort="${X4_moderate_effort}" velocity="${X4_rated_velocity}" lower="-0.79" upper="0.79"/>
-    <dynamics friction="${X4_friction}" damping="${X4_damping}"/>
+    <limit effort="${X4_moderate_effort}" velocity="${X4_rated_velocity}" lower="-0.785398" upper="0.785398"/>
+    <dynamics damping="${X4_damping}" friction="${X4_friction}"/>
   </joint>
 </robot>

File: ldr-harambe-v0.4/urdf/joints/right_arm_joints.xacro (robot description, xacro)
@@ -9,6 +9,6 @@
     <child link="urdf_r_shoulder_assembly"/>
     <axis xyz="0 1 0"/>
-    <limit effort="${X6_moderate_effort}" velocity="${X6_rated_velocity}" lower="-3.02" upper="1.69"/>
-    <dynamics friction="${X6_friction}" damping="${X6_damping}"/>
+    <limit effort="${X6_moderate_effort}" velocity="${X6_rated_velocity}" lower="-3.01942" upper="1.69297"/>
+    <dynamics damping="${X6_damping}" friction="${X6_friction}"/>
   </joint>
   <joint name="right_shoulder_roll_joint_X6" type="revolute">
@@ -17,6 +17,6 @@
     <child link="urdf_r_upper_arm_assembly"/>
     <axis xyz="1 0 0"/>
-    <limit effort="${X6_moderate_effort}" velocity="${X6_rated_velocity}" lower="-2.93" upper="0.21"/>
-    <dynamics friction="${X6_friction}" damping="${X6_damping}"/>
+    <limit effort="${X6_moderate_effort}" velocity="${X6_rated_velocity}" lower="-2.93215" upper="0.20944"/>
+    <dynamics damping="${X6_damping}" friction="${X6_friction}"/>
   </joint>
   <joint name="right_shoulder_yaw_joint_X4" type="revolute">
@@ -25,6 +25,6 @@
     <child link="urdf_r_elbow_assembly"/>
     <axis xyz="0 0 1"/>
-    <limit effort="${X4_moderate_effort}" velocity="${X4_rated_velocity}" lower="-2.97" upper="1.75"/>
-    <dynamics friction="${X4_friction}" damping="${X4_damping}"/>
+    <limit effort="${X4_moderate_effort}" velocity="${X4_rated_velocity}" lower="-2.96706" upper="1.74533"/>
+    <dynamics damping="${X4_damping}" friction="${X4_friction}"/>
   </joint>
   <joint name="right_elbow_pitch_joint_X6" type="revolute">
@@ -33,6 +33,6 @@
     <child link="urdf_r_upper_forearm_assembly"/>
     <axis xyz="0 1 0"/>
-    <limit effort="${X6_moderate_effort}" velocity="${X6_rated_velocity}" lower="-1.31" upper="1.83"/>
-    <dynamics friction="${X6_friction}" damping="${X6_damping}"/>
+    <limit effort="${X6_moderate_effort}" velocity="${X6_rated_velocity}" lower="-1.309" upper="1.8326"/>
+    <dynamics damping="${X6_damping}" friction="${X6_friction}"/>
   </joint>
   <joint name="right_wrist_yaw_joint_X4" type="revolute">
@@ -41,6 +41,6 @@
     <child link="urdf_r_lower_forearm_assembly"/>
     <axis xyz="0 0 1"/>
-    <limit effort="${X4_moderate_effort}" velocity="${X4_rated_velocity}" lower="-2.36" upper="2.36"/>
-    <dynamics friction="${X4_friction}" damping="${X4_damping}"/>
+    <limit effort="${X4_moderate_effort}" velocity="${X4_rated_velocity}" lower="-2.35619" upper="2.35619"/>
+    <dynamics damping="${X4_damping}" friction="${X4_friction}"/>
   </joint>
   <joint name="right_wrist_roll_joint_X4" type="revolute">
@@ -49,6 +49,6 @@
     <child link="urdf_r_wrist_assembly"/>
     <axis xyz="1 0 0"/>
-    <limit effort="${X4_moderate_effort}" velocity="${X4_rated_velocity}" lower="-1.57" upper="1.57"/>
-    <dynamics friction="${X4_friction}" damping="${X4_damping}"/>
+    <limit effort="${X4_moderate_effort}" velocity="${X4_rated_velocity}" lower="-1.65806" upper="1.65806"/>
+    <dynamics damping="${X4_damping}" friction="${X4_friction}"/>
   </joint>
 </robot>

File: ldr-harambe-v0.4/urdf/joints/right_foot_joints.xacro (robot description, xacro)
@@ -9,6 +9,6 @@
     <child link="urdf_hip_assembly_2"/>
     <axis xyz="0 1 0"/>
-    <limit effort="${X8_moderate_effort}" velocity="${X8_rated_velocity}" lower="-2.53" upper="1.57"/>
-    <dynamics friction="${X8_friction}" damping="${X8_damping}"/>
+    <limit effort="${X8_moderate_effort}" velocity="${X8_rated_velocity}" lower="-2.61799" upper="2.61799"/>
+    <dynamics damping="${X8_damping}" friction="${X8_friction}"/>
   </joint>
   <joint name="right_hip_roll_joint_X8" type="${leg_joint_type}">
@@ -17,6 +17,6 @@
     <child link="urdf_r_upper_femur_assemby"/>
     <axis xyz="1 0 0"/>
-    <limit effort="${X8_moderate_effort}" velocity="${X8_rated_velocity}" lower="-3.14" upper="0.35"/>
-    <dynamics friction="${X8_friction}" damping="${X8_damping}"/>
+    <limit effort="${X8_moderate_effort}" velocity="${X8_rated_velocity}" lower="-3.22886" upper="0.383972"/>
+    <dynamics damping="${X8_damping}" friction="${X8_friction}"/>
   </joint>
   <joint name="right_hip_yaw_joint_X8" type="${leg_joint_type}">
@@ -25,6 +25,6 @@
     <child link="urdf_lower_femur_assembly_2"/>
     <axis xyz="0 0 1"/>
-    <limit effort="${X8_moderate_effort}" velocity="${X8_rated_velocity}" lower="-1.57" upper="1.57"/>
-    <dynamics friction="${X8_friction}" damping="${X8_damping}"/>
+    <limit effort="${X8_moderate_effort}" velocity="${X8_rated_velocity}" lower="-1.5708" upper="1.5708"/>
+    <dynamics damping="${X8_damping}" friction="${X8_friction}"/>
   </joint>
   <joint name="right_knee_joint_X8" type="${leg_joint_type}">
@@ -33,6 +33,6 @@
     <child link="urdf_r_tibia_assembly"/>
     <axis xyz="0 1 0"/>
-    <limit effort="${X8_moderate_effort}" velocity="${X8_rated_velocity}" lower="-0.17" upper="1.57"/>
-    <dynamics friction="${X8_friction}" damping="${X8_damping}"/>
+    <limit effort="${X8_moderate_effort}" velocity="${X8_rated_velocity}" lower="-1.52716" upper="1.52716"/>
+    <dynamics damping="${X8_damping}" friction="${X8_friction}"/>
   </joint>
   <joint name="right_ankle_roll_joint_X4" type="${leg_joint_type}">
@@ -41,6 +41,6 @@
     <child link="udrf_ankle_assembly_2"/>
     <axis xyz="1 0 0"/>
-    <limit effort="${X4_moderate_effort}" velocity="${X4_rated_velocity}" lower="-0.79" upper="0.79"/>
-    <dynamics friction="${X4_friction}" damping="${X4_damping}"/>
+    <limit effort="${X4_moderate_effort}" velocity="${X4_rated_velocity}" lower="-0.785398" upper="0.785398"/>
+    <dynamics damping="${X4_damping}" friction="${X4_friction}"/>
   </joint>
   <joint name="right_ankle_pitch_joint_X4" type="${leg_joint_type}">
@@ -49,6 +49,6 @@
     <child link="urdf_foot_assembly_2"/>
     <axis xyz="0 1 0"/>
-    <limit effort="${X4_moderate_effort}" velocity="${X4_rated_velocity}" lower="-0.79" upper="0.79"/>
-    <dynamics friction="${X4_friction}" damping="${X4_damping}"/>
+    <limit effort="${X4_moderate_effort}" velocity="${X4_rated_velocity}" lower="-0.785398" upper="0.785398"/>
+    <dynamics damping="${X4_damping}" friction="${X4_friction}"/>
   </joint>
 </robot>
