Commit message: ankle axes correction harambe v0.4

File: ldr-harambe-v0.4/robot_harambe_v04.urdf (robot description, URDF)
Before this commit: robot robot_harambe_v04, 26 links, 25 joints
Joints:
- joint right_ankle_pitch_joint_X4: child urdf_foot_assembly_2 -> udrf_ankle_assembly_2; origin xyz=-0.012 0.028 -0.004 rpy=0 1.5708 0 -> xyz=-0 0.395 0.059 rpy=0 -0 -0; parent udrf_ankle_assembly_2 -> urdf_r_tibia_assembly
- joint right_ankle_roll_joint_X4: child udrf_ankle_assembly_2 -> urdf_foot_assembly_2; origin xyz=-0 0.395 0.059 rpy=0 -0 -0 -> xyz=-0.012 0.028 -0.004 rpy=0 1.5708 0; parent urdf_r_tibia_assembly -> udrf_ankle_assembly_2

File: ldr-harambe-v0.4/robot_harambe_v04_fixed_axes.urdf (robot description, URDF)
Before this commit: robot robot_harambe_v04, 26 links, 25 joints
Joints:
- joint right_ankle_pitch_joint_X4: axis 1 0 0 -> 0 1 0
- joint right_ankle_roll_joint_X4: axis 0 1 0 -> 1 0 0

File: ldr-harambe-v0.4/robot_harambe_v04_fixed_axes_limits.urdf (robot description, URDF)
Before this commit: robot robot_harambe_v04, 26 links, 25 joints
Joints:
- joint right_ankle_pitch_joint_X4: axis 1 0 0 -> 0 1 0
- joint right_ankle_roll_joint_X4: axis 0 1 0 -> 1 0 0

File: ldr-harambe-v0.4/robot_harambe_v04_fixed_axes_limits_simplified.urdf (robot description, URDF)
Before this commit: robot robot_harambe_v04, 26 links, 25 joints
Joints:
- joint right_ankle_pitch_joint_X4: axis 1 0 0 -> 0 1 0
- joint right_ankle_roll_joint_X4: axis 0 1 0 -> 1 0 0

File: ldr-harambe-v0.4/robot_harambe_v04_fixed_axes_limits_simplified_no_collision.urdf (robot description, URDF)
Before this commit: robot robot_harambe_v04, 26 links, 25 joints
Joints:
- joint right_ankle_pitch_joint_X4: axis 1 0 0 -> 0 1 0
- joint right_ankle_roll_joint_X4: axis 0 1 0 -> 1 0 0

Commit message: mass correction

File: ldr-harambe-v0.4/robot_harambe_v04.urdf (robot description, URDF)
Before this commit: robot robot_harambe_v04, 26 links, 25 joints
Links:
- link urdf_foot_assembly: mass 309 -> 0.309
- link urdf_foot_assembly_2: mass 309 -> 0.309

File: ldr-harambe-v0.4/robot_harambe_v04_fixed_axes.urdf (robot description, URDF)
Before this commit: robot robot_harambe_v04, 26 links, 25 joints
Links:
- link urdf_foot_assembly: mass 309 -> 0.309
- link urdf_foot_assembly_2: mass 309 -> 0.309

File: ldr-harambe-v0.4/robot_harambe_v04_fixed_axes_limits.urdf (robot description, URDF)
Before this commit: robot robot_harambe_v04, 26 links, 25 joints
Links:
- link urdf_foot_assembly: mass 309 -> 0.309
- link urdf_foot_assembly_2: mass 309 -> 0.309

File: ldr-harambe-v0.4/robot_harambe_v04_fixed_axes_limits_simplified.urdf (robot description, URDF)
Before this commit: robot robot_harambe_v04, 26 links, 25 joints
Links:
- link urdf_foot_assembly: mass 309 -> 0.309
- link urdf_foot_assembly_2: mass 309 -> 0.309

File: ldr-harambe-v0.4/robot_harambe_v04_fixed_axes_limits_simplified_no_collision.urdf (robot description, URDF)
Before this commit: robot robot_harambe_v04, 26 links, 25 joints
Links:
- link urdf_foot_assembly: mass 309 -> 0.309
- link urdf_foot_assembly_2: mass 309 -> 0.309

Commit message: typo review

File: ldr-harambe-v0.4/robot_harambe_v04.urdf (robot description, URDF)
Before this commit: robot robot_harambe_v04, 26 links, 25 joints
Links:
- removed link udrf_ankle_assembly
- removed link udrf_ankle_assembly_2
- added link urdf_ankle_assembly, mass 0.0818219; collision mesh filename=package://assets/urdf_ankle_assembly.stl; visual mesh filename=package://assets/urdf_ankle_assembly.stl
- added link urdf_ankle_assembly_2, mass 0.0818219; collision mesh filename=package://assets/urdf_ankle_assembly.stl; visual mesh filename=package://assets/urdf_ankle_assembly.stl
Joints:
- joint left_ankle_pitch_joint_X4: child udrf_ankle_assembly -> urdf_ankle_assembly
- joint left_ankle_roll_joint_X4: parent udrf_ankle_assembly -> urdf_ankle_assembly
- joint right_ankle_pitch_joint_X4: child udrf_ankle_assembly_2 -> urdf_ankle_assembly_2
- joint right_ankle_roll_joint_X4: parent udrf_ankle_assembly_2 -> urdf_ankle_assembly_2

File: ldr-harambe-v0.4/robot_harambe_v04_fixed_axes.urdf (robot description, URDF)
Before this commit: robot robot_harambe_v04, 26 links, 25 joints
Links:
- removed link udrf_ankle_assembly
- removed link udrf_ankle_assembly_2
- added link urdf_ankle_assembly, mass 0.0818219; collision mesh filename=package://assets/urdf_ankle_assembly.stl; visual mesh filename=package://assets/urdf_ankle_assembly.stl
- added link urdf_ankle_assembly_2, mass 0.0818219; collision mesh filename=package://assets/urdf_ankle_assembly.stl; visual mesh filename=package://assets/urdf_ankle_assembly.stl
Joints:
- joint left_ankle_pitch_joint_X4: child udrf_ankle_assembly -> urdf_ankle_assembly
- joint left_ankle_roll_joint_X4: parent udrf_ankle_assembly -> urdf_ankle_assembly
- joint right_ankle_pitch_joint_X4: parent udrf_ankle_assembly_2 -> urdf_ankle_assembly_2
- joint right_ankle_roll_joint_X4: child udrf_ankle_assembly_2 -> urdf_ankle_assembly_2

File: ldr-harambe-v0.4/robot_harambe_v04_fixed_axes_simplified.urdf (robot description, URDF)
Before this commit: robot robot_harambe_v04, 26 links, 25 joints
Links:
- removed link udrf_ankle_assembly
- removed link udrf_ankle_assembly_2
- added link urdf_ankle_assembly, mass 0.0818219; collision mesh filename=package://meshes/collision/urdf_ankle_assembly.stl; visual mesh filename=package://meshes/visual/urdf_ankle_assembly.stl
- added link urdf_ankle_assembly_2, mass 0.0818219; collision mesh filename=package://meshes/collision/urdf_ankle_assembly.stl; visual mesh filename=package://meshes/visual/urdf_ankle_assembly.stl
Joints:
- joint left_ankle_pitch_joint_X4: child udrf_ankle_assembly -> urdf_ankle_assembly
- joint left_ankle_roll_joint_X4: parent udrf_ankle_assembly -> urdf_ankle_assembly
- joint right_ankle_pitch_joint_X4: parent udrf_ankle_assembly_2 -> urdf_ankle_assembly_2
- joint right_ankle_roll_joint_X4: child udrf_ankle_assembly_2 -> urdf_ankle_assembly_2

File: ldr-harambe-v0.4/robot_harambe_v04_fixed_axes_simplified_no_collision.urdf (robot description, URDF)
Before this commit: robot robot_harambe_v04, 26 links, 25 joints
Links:
- removed link udrf_ankle_assembly
- removed link udrf_ankle_assembly_2
- added link urdf_ankle_assembly, mass 0.0818219; collision mesh filename=package://meshes/collision/urdf_ankle_assembly.stl; visual mesh filename=package://meshes/visual/urdf_ankle_assembly.stl
- added link urdf_ankle_assembly_2, mass 0.0818219; collision mesh filename=package://meshes/collision/urdf_ankle_assembly.stl; visual mesh filename=package://meshes/visual/urdf_ankle_assembly.stl
Joints:
- joint left_ankle_pitch_joint_X4: child udrf_ankle_assembly -> urdf_ankle_assembly
- joint left_ankle_roll_joint_X4: parent udrf_ankle_assembly -> urdf_ankle_assembly
- joint right_ankle_pitch_joint_X4: parent udrf_ankle_assembly_2 -> urdf_ankle_assembly_2
- joint right_ankle_roll_joint_X4: child udrf_ankle_assembly_2 -> urdf_ankle_assembly_2

File: ldr-harambe-v0.4/urdf/joints/left_foot_joints.xacro (robot description, xacro)
@@ -39,5 +39,5 @@
     <origin xyz="0 -0.051 -0.395" rpy="0 0 0"/>
     <parent link="urdf_l_tibia_assembly"/>
-    <child link="udrf_ankle_assembly"/>
+    <child link="urdf_ankle_assembly"/>
     <axis xyz="0 1 0"/>
     <limit effort="${X4_moderate_effort}" velocity="${X4_rated_velocity}" lower="-0.785398" upper="0.785398"/>
@@ -46,5 +46,5 @@
   <joint name="left_ankle_roll_joint_X4" type="${leg_joint_type}">
     <origin xyz="-0.012 -0.004 -0.028" rpy="0 0 0"/>
-    <parent link="udrf_ankle_assembly"/>
+    <parent link="urdf_ankle_assembly"/>
     <child link="urdf_foot_assembly"/>
     <axis xyz="1 0 0"/>

File: ldr-harambe-v0.4/urdf/joints/right_foot_joints.xacro (robot description, xacro)
@@ -39,5 +39,5 @@
     <origin xyz="0 0.059 -0.395" rpy="0 0 0"/>
     <parent link="urdf_r_tibia_assembly"/>
-    <child link="udrf_ankle_assembly_2"/>
+    <child link="urdf_ankle_assembly_2"/>
     <axis xyz="0 1 0"/>
     <limit effort="${X4_moderate_effort}" velocity="${X4_rated_velocity}" lower="-0.79" upper="0.79"/>
@@ -46,5 +46,5 @@
   <joint name="right_ankle_roll_joint_X4" type="${leg_joint_type}">
     <origin xyz="-0.012 -0.004 -0.028" rpy="0 0 0"/>
-    <parent link="udrf_ankle_assembly_2"/>
+    <parent link="urdf_ankle_assembly_2"/>
     <child link="urdf_foot_assembly_2"/>
     <axis xyz="1 0 0"/>

File: ldr-harambe-v0.4/urdf/links/left_foot_links.xacro (robot description, xacro)
@@ -203,5 +203,5 @@
     </visual>
   </link>
-  <link name="udrf_ankle_assembly">
+  <link name="urdf_ankle_assembly">
     <inertial>
       <origin xyz="0 -0.004 -0.0125426" rpy="0 0 0"/>
@@ -212,7 +212,7 @@
       <origin xyz="0 -0.004 -0.0125426" rpy="0 0 -1.5708"/>
       <geometry>
-        <mesh filename="package://full_robot_description/meshes/visual/udrf_ankle_assembly.stl"/>
-      </geometry>
-      <material name="udrf_ankle_assembly_material">
+        <mesh filename="package://full_robot_description/meshes/visual/urdf_ankle_assembly.stl"/>
+      </geometry>
+      <material name="urdf_ankle_assembly_material">
         <color rgba="0.615686 0.811765 0.929412 1"/>
       </material>
@@ -221,5 +221,5 @@
       <origin xyz="0 -0.004 -0.0125426" rpy="0 0 -1.5708"/>
       <geometry>
-        <mesh filename="package://full_robot_description/meshes/collision/udrf_ankle_assembly.stl"/>
+        <mesh filename="package://full_robot_description/meshes/collision/urdf_ankle_assembly.stl"/>
       </geometry>
     </collision>

File: ldr-harambe-v0.4/urdf/links/right_foot_links.xacro (robot description, xacro)
@@ -173,5 +173,5 @@
     </visual>
   </link>
-  <link name="udrf_ankle_assembly_2">
+  <link name="urdf_ankle_assembly_2">
     <inertial>
       <origin xyz="0 -0.004 -0.0125426" rpy="0 0 0"/>
@@ -182,7 +182,7 @@
       <origin xyz="0 -0.004 -0.0125426" rpy="0 0 -1.5708"/>
       <geometry>
-        <mesh filename="package://full_robot_description/meshes/visual/udrf_ankle_assembly.stl"/>
-      </geometry>
-      <material name="udrf_ankle_assembly_2_material">
+        <mesh filename="package://full_robot_description/meshes/visual/urdf_ankle_assembly.stl"/>
+      </geometry>
+      <material name="urdf_ankle_assembly_2_material">
         <color rgba="0.615686 0.811765 0.929412 1"/>
       </material>
@@ -191,5 +191,5 @@
       <origin xyz="0 -0.004 -0.0125426" rpy="0 0 -1.5708"/>
       <geometry>
-        <mesh filename="package://full_robot_description/meshes/collision/udrf_ankle_assembly.stl"/>
+        <mesh filename="package://full_robot_description/meshes/collision/urdf_ankle_assembly.stl"/>
       </geometry>
     </collision>
