Commit message: correction splited urdf

File: ldr-harambe-v0.4/urdf/joints/right_foot_joints.xacro (robot description, xacro)
@@ -40,5 +40,5 @@
     <parent link="urdf_r_tibia_assembly"/>
     <child link="udrf_ankle_assembly_2"/>
-    <axis xyz="0 1 0"/>
+    <axis xyz="1 0 0"/>
     <limit effort="${X4_moderate_effort}" velocity="${X4_rated_velocity}" lower="-0.79" upper="0.79"/>
     <dynamics friction="${X4_friction}" damping="${X4_damping}"/>
@@ -48,5 +48,5 @@
     <parent link="udrf_ankle_assembly_2"/>
     <child link="urdf_foot_assembly_2"/>
-    <axis xyz="1 0 0"/>
+    <axis xyz="0 1 0"/>
     <limit effort="${X4_moderate_effort}" velocity="${X4_rated_velocity}" lower="-0.79" upper="0.79"/>
     <dynamics friction="${X4_friction}" damping="${X4_damping}"/>

File: ldr-harambe-v0.4/urdf/links/left_foot_links.xacro (robot description, xacro)
@@ -228,6 +228,6 @@
     <inertial>
       <origin xyz="0.0436027 8.11114e-08 -0.0200314" rpy="0 0 0"/>
-      <mass value="309"/>
-      <inertia ixx="0.232433" ixy="-1.58776e-08" ixz="-0.00983566" iyy="1.21361" iyz="-6.57666e-07" izz="1.37693"/>
+      <mass value="0.309"/>
+      <inertia ixx="0.000232433" ixy="-1.58776e-11" ixz="-9.83566e-06" iyy="0.00121361" iyz="-6.57666e-10" izz="0.00137693"/>
     </inertial>
     <visual>

File: ldr-harambe-v0.4/urdf/links/right_foot_links.xacro (robot description, xacro)
@@ -198,6 +198,6 @@
     <inertial>
       <origin xyz="0.0436027 8.11114e-08 -0.0200314" rpy="0 0 0"/>
-      <mass value="309"/>
-      <inertia ixx="0.232433" ixy="-1.58776e-08" ixz="-0.00983566" iyy="1.21361" iyz="-6.57666e-07" izz="1.37693"/>
+      <mass value="0.309"/>
+      <inertia ixx="0.000232433" ixy="-1.58776e-11" ixz="-9.83566e-06" iyy="0.00121361" iyz="-6.57666e-10" izz="0.00137693"/>
     </inertial>
     <visual>

Commit message: right ankle order correction

File: ldr-harambe-v0.4/urdf/joints/right_foot_joints.xacro (robot description, xacro)
@@ -36,19 +36,19 @@
     <dynamics damping="${X8_damping}" friction="${X8_friction}"/>
   </joint>
-  <joint name="right_ankle_roll_joint_X4" type="${leg_joint_type}">
+  <joint name="right_ankle_pitch_joint_X4" type="${leg_joint_type}">
     <origin xyz="0 0.059 -0.395" rpy="0 0 0"/>
     <parent link="urdf_r_tibia_assembly"/>
     <child link="udrf_ankle_assembly_2"/>
-    <axis xyz="1 0 0"/>
-    <limit effort="${X4_moderate_effort}" velocity="${X4_rated_velocity}" lower="-0.785398" upper="0.785398"/>
-    <dynamics damping="${X4_damping}" friction="${X4_friction}"/>
+    <axis xyz="0 1 0"/>
+    <limit effort="${X4_moderate_effort}" velocity="${X4_rated_velocity}" lower="-0.79" upper="0.79"/>
+    <dynamics friction="${X4_friction}" damping="${X4_damping}"/>
   </joint>
-  <joint name="right_ankle_pitch_joint_X4" type="${leg_joint_type}">
+  <joint name="right_ankle_roll_joint_X4" type="${leg_joint_type}">
     <origin xyz="-0.012 -0.004 -0.028" rpy="0 0 0"/>
     <parent link="udrf_ankle_assembly_2"/>
     <child link="urdf_foot_assembly_2"/>
-    <axis xyz="0 1 0"/>
-    <limit effort="${X4_moderate_effort}" velocity="${X4_rated_velocity}" lower="-0.785398" upper="0.785398"/>
-    <dynamics damping="${X4_damping}" friction="${X4_friction}"/>
+    <axis xyz="1 0 0"/>
+    <limit effort="${X4_moderate_effort}" velocity="${X4_rated_velocity}" lower="-0.79" upper="0.79"/>
+    <dynamics friction="${X4_friction}" damping="${X4_damping}"/>
   </joint>
 </robot>
