Commit message: harambe v0.4 origin pervis base

File: ldr-harambe-V0.4-com2origin/robot_harambe_v04_com2origin.urdf (robot description, URDF)
Before this commit: robot robot_harambe_v04_com2origin, 26 links, 25 joints
Links:
- removed link urdf_base
- added link urdf_pelvis, mass 5.778; collision mesh filename=package://assets/urdf_pelvis.stl; visual mesh filename=package://assets/urdf_pelvis.stl
Joints:
- joint left_ankle_pitch_joint_X4: origin xyz=0 0.395 -0.051 rpy=0 0 -0 -> xyz=-0 0.395 -0.051 rpy=0 0 -0
- joint left_hip_pitch_joint_X8: parent urdf_base -> urdf_pelvis
- joint left_hip_roll_joint_X8: origin xyz=0 -0.053 -0.062 rpy=1.5708 -1.5708 0 -> xyz=-0 -0.053 -0.062 rpy=1.5708 -1.5708 0
- joint right_hip_pitch_joint_X8: parent urdf_base -> urdf_pelvis
- joint right_wrist_roll_joint_X4: origin xyz=-0 -0.033 0.0565 rpy=1.5708 -0 0 -> xyz=0 -0.033 0.0565 rpy=1.5708 -0 0
- joint waist_yaw_joint_X8: parent urdf_base -> urdf_pelvis

Commit message: format

File: ldr-harambe-V0.4-com2origin/robot_harambe_v04_com2origin.urdf (robot description, URDF)
Before this commit: robot robot_harambe_v04_com2origin, 26 links, 25 joints
Links:
- removed link urdf_pelvis
- added link urdf_base, mass 5.778; collision mesh filename=package://assets/urdf_base.stl; visual mesh filename=package://assets/urdf_base.stl
Joints:
- joint left_hip_pitch_joint_X8: parent urdf_pelvis -> urdf_base
- joint right_hip_pitch_joint_X8: parent urdf_pelvis -> urdf_base
- joint waist_yaw_joint_X8: parent urdf_pelvis -> urdf_base

File: ldr-harambe-V0.4-com2origin/robot_harambe_v04_com2origin_fixed_axes.urdf (robot description, URDF)
Before this commit: robot robot_harambe_v04_com2origin, 26 links, 25 joints
Links:
- link urdf_base: geometry collision mesh filename=package://assets/urdf_base.stl; visual mesh filename=package://assets/urdf_base.stl

File: ldr-harambe-V0.4-com2origin/robot_harambe_v04_com2origin_fixed_axes_simplified.urdf (robot description, URDF)
Before this commit: robot robot_harambe_v04_com2origin, 26 links, 25 joints
Links:
- link urdf_base: geometry collision mesh filename=package://meshes/collision/urdf_base.stl; visual mesh filename=package://meshes/visual/urdf_base.stl

File: ldr-harambe-V0.4-com2origin/robot_harambe_v04_com2origin_fixed_axes_simplified_no_collision.urdf (robot description, URDF)
Before this commit: robot robot_harambe_v04_com2origin, 26 links, 25 joints
Links:
- link urdf_base: geometry collision mesh filename=package://meshes/collision/urdf_base.stl; visual mesh filename=package://meshes/visual/urdf_base.stl

File: ldr-harambe-V0.4-com2origin/urdf/links/body_links.xacro (robot description, xacro)
@@ -6,62 +6,14 @@
   <link name="urdf_base">
     <inertial>
-      <origin xyz="-0.0140423 0.000165152 -0.0361968" rpy="0 0 0"/>
+      <origin xyz="-0.0133337 0.000163695 -0.0360702" rpy="0 0 0"/>
       <mass value="5.778"/>
-      <inertia ixx="0.0290802" ixy="1.02817e-06" ixz="7.34969e-05" iyy="0.0242074" iyz="-1.43152e-05" izz="0.0161172"/>
+      <inertia ixx="0.0319377" ixy="1.97277e-06" ixz="3.91267e-05" iyy="0.0280522" iyz="-4.94971e-07" izz="0.0192445"/>
     </inertial>
-    <visual>
-      <origin xyz="-0.015194 -0.00383235 -0.0706295" rpy="0 -1.57079 1.5708"/>
-      <geometry>
-        <mesh filename="package://full_robot_description/meshes/visual/stator_x8_p20_120_unified.stl"/>
-      </geometry>
-      <material name="stator_x8_p20_120_unified_material">
-        <color rgba="0.882353 0.572549 0.478431 1"/>
-      </material>
-    </visual>
     <visual>
       <origin xyz="-0.015194 0.000167649 -0.0706295" rpy="0 0 -1.5708"/>
       <geometry>
-        <mesh filename="package://full_robot_description/meshes/visual/b_base.stl"/>
+        <mesh filename="package://full_robot_description/meshes/visual/urdf_base.stl"/>
       </geometry>
-      <material name="b_base_material">
-        <color rgba="0.980392 0.713725 0.00392157 1"/>
-      </material>
-    </visual>
-    <collision>
-      <origin xyz="-0.015194 0.000167649 -0.0706295" rpy="0 0 -1.5708"/>
-      <geometry>
-        <mesh filename="package://full_robot_description/meshes/collision/b_base.stl"/>
-      </geometry>
-    </collision>
-    <visual>
-      <origin xyz="-0.015194 0.000167649 -0.0706295" rpy="-3.14159 0 -1.5708"/>
-      <geometry>
-        <mesh filename="package://full_robot_description/meshes/visual/plate_base_right.stl"/>
-      </geometry>
-      <material name="plate_base_right_material">
-        <color rgba="0.654902 0.823529 0.576471 1"/>
-      </material>
-    </visual>
-    <collision>
-      <origin xyz="-0.015194 0.000167649 -0.0706295" rpy="-3.14159 0 -1.5708"/>
-      <geometry>
-        <mesh filename="package://full_robot_description/meshes/collision/plate_base_right.stl"/>
-      </geometry>
-    </collision>
-    <visual>
-      <origin xyz="-0.015194 0.000167649 0.20937" rpy="-3.14159 0 -1.5708"/>
-      <geometry>
-        <mesh filename="package://full_robot_description/meshes/visual/spacer_pelvis_torso.stl"/>
-      </geometry>
-      <material name="spacer_pelvis_torso_material">
-        <color rgba="0.498039 0.498039 0.498039 1"/>
-      </material>
-    </visual>
-    <visual>
-      <origin xyz="-0.015194 0.000167649 -0.0706295" rpy="0 0 -1.5708"/>
-      <geometry>
-        <mesh filename="package://full_robot_description/meshes/visual/f_base.stl"/>
-      </geometry>
-      <material name="f_base_material">
+      <material name="urdf_base_material">
         <color rgba="0.231373 0.380392 0.705882 1"/>
       </material>
@@ -70,83 +22,5 @@
       <origin xyz="-0.015194 0.000167649 -0.0706295" rpy="0 0 -1.5708"/>
       <geometry>
-        <mesh filename="package://full_robot_description/meshes/collision/f_base.stl"/>
-      </geometry>
-    </collision>
-    <visual>
-      <origin xyz="-0.015194 0.000167649 -0.0706295" rpy="0 0 -1.5708"/>
-      <geometry>
-        <mesh filename="package://full_robot_description/meshes/visual/cap_b_base.stl"/>
-      </geometry>
-      <material name="cap_b_base_material">
-        <color rgba="0.596078 0.121569 0.67451 1"/>
-      </material>
-    </visual>
-    <collision>
-      <origin xyz="-0.015194 0.000167649 -0.0706295" rpy="0 0 -1.5708"/>
-      <geometry>
-        <mesh filename="package://full_robot_description/meshes/collision/cap_b_base.stl"/>
-      </geometry>
-    </collision>
-    <visual>
-      <origin xyz="-0.015194 0.000167649 -0.00462952" rpy="0 0 -1.5708"/>
-      <geometry>
-        <mesh filename="package://full_robot_description/meshes/visual/stator_x8_p20_120_unified.stl"/>
-      </geometry>
-      <material name="stator_x8_p20_120_unified_2_material">
-        <color rgba="0.882353 0.572549 0.478431 1"/>
-      </material>
-    </visual>
-    <visual>
-      <origin xyz="-0.015194 0.000167649 -0.0706295" rpy="0 0 -1.5708"/>
-      <geometry>
-        <mesh filename="package://full_robot_description/meshes/visual/plate_base_left.stl"/>
-      </geometry>
-      <material name="plate_base_left_material">
-        <color rgba="0.764706 0.545098 0.803922 1"/>
-      </material>
-    </visual>
-    <collision>
-      <origin xyz="-0.015194 0.000167649 -0.0706295" rpy="0 0 -1.5708"/>
-      <geometry>
-        <mesh filename="package://full_robot_description/meshes/collision/plate_base_left.stl"/>
-      </geometry>
-    </collision>
-    <visual>
-      <origin xyz="-0.015194 0.000167649 -0.0706295" rpy="0 0 -1.5708"/>
-      <geometry>
-        <mesh filename="package://full_robot_description/meshes/visual/plate_base_top.stl"/>
-      </geometry>
-      <material name="plate_base_top_material">
-        <color rgba="0.654902 0.584314 0.823529 1"/>
-      </material>
-    </visual>
-    <collision>
-      <origin xyz="-0.015194 0.000167649 -0.0706295" rpy="0 0 -1.5708"/>
-      <geometry>
-        <mesh filename="package://full_robot_description/meshes/collision/plate_base_top.stl"/>
-      </geometry>
-    </collision>
-    <visual>
-      <origin xyz="-0.015194 0.00416765 -0.0706295" rpy="0 1.57079 1.5708"/>
-      <geometry>
-        <mesh filename="package://full_robot_description/meshes/visual/stator_x8_p20_120_unified.stl"/>
-      </geometry>
-      <material name="stator_x8_p20_120_unified_3_material">
-        <color rgba="0.882353 0.572549 0.478431 1"/>
-      </material>
-    </visual>
-    <visual>
-      <origin xyz="-0.015194 0.000167649 -0.0706295" rpy="0 0 -1.5708"/>
-      <geometry>
-        <mesh filename="package://full_robot_description/meshes/visual/jockstrap.stl"/>
-      </geometry>
-      <material name="jockstrap_material">
-        <color rgba="0.615686 0.811765 0.929412 1"/>
-      </material>
-    </visual>
-    <collision>
-      <origin xyz="-0.015194 0.000167649 -0.0706295" rpy="0 0 -1.5708"/>
-      <geometry>
-        <mesh filename="package://full_robot_description/meshes/collision/jockstrap.stl"/>
+        <mesh filename="package://full_robot_description/meshes/collision/urdf_base.stl"/>
       </geometry>
     </collision>

File: ldr-harambe-V0.4-com2origin/urdf/links/left_foot_links.xacro (robot description, xacro)
@@ -30,5 +30,5 @@
         <mesh filename="package://full_robot_description/meshes/visual/stator_x8_p20_120_unified.stl"/>
       </geometry>
-      <material name="stator_x8_p20_120_unified_4_material">
+      <material name="stator_x8_p20_120_unified_material">
         <color rgba="0.882353 0.572549 0.478431 1"/>
       </material>
@@ -76,5 +76,5 @@
         <mesh filename="package://full_robot_description/meshes/visual/stator_x8_p20_120_unified.stl"/>
       </geometry>
-      <material name="stator_x8_p20_120_unified_5_material">
+      <material name="stator_x8_p20_120_unified_2_material">
         <color rgba="0.882353 0.572549 0.478431 1"/>
       </material>
@@ -122,5 +122,5 @@
         <mesh filename="package://full_robot_description/meshes/visual/stator_x8_p20_120_unified.stl"/>
       </geometry>
-      <material name="stator_x8_p20_120_unified_6_material">
+      <material name="stator_x8_p20_120_unified_3_material">
         <color rgba="0.882353 0.572549 0.478431 1"/>
       </material>

File: ldr-harambe-V0.4-com2origin/urdf/links/right_foot_links.xacro (robot description, xacro)
@@ -30,5 +30,5 @@
         <mesh filename="package://full_robot_description/meshes/visual/stator_x8_p20_120_unified.stl"/>
       </geometry>
-      <material name="stator_x8_p20_120_unified_7_material">
+      <material name="stator_x8_p20_120_unified_4_material">
         <color rgba="0.882353 0.572549 0.478431 1"/>
       </material>
@@ -61,5 +61,5 @@
         <mesh filename="package://full_robot_description/meshes/visual/stator_x8_p20_120_unified.stl"/>
       </geometry>
-      <material name="stator_x8_p20_120_unified_8_material">
+      <material name="stator_x8_p20_120_unified_5_material">
         <color rgba="0.882353 0.572549 0.478431 1"/>
       </material>
@@ -92,5 +92,5 @@
         <mesh filename="package://full_robot_description/meshes/visual/stator_x8_p20_120_unified.stl"/>
       </geometry>
-      <material name="stator_x8_p20_120_unified_9_material">
+      <material name="stator_x8_p20_120_unified_6_material">
         <color rgba="0.882353 0.572549 0.478431 1"/>
       </material>
