Commit message: multiple corrections

File: ldr-harambe-V0.4-com2origin/robot_harambe_v04_com2origin.urdf (robot description, URDF)
Before this commit: robot robot_harambe_v04_com2origin, 26 links, 25 joints
Links:
- removed link udrf_ankle_assembly
- removed link udrf_ankle_assembly_2
- removed link urdf_r_upper_femur_assemby
- added link urdf_ankle_assembly, mass 0.0818219; collision mesh filename=package://assets/urdf_ankle_assembly.stl; visual mesh filename=package://assets/urdf_ankle_assembly.stl
- added link urdf_ankle_assembly_2, mass 0.0818219; collision mesh filename=package://assets/urdf_ankle_assembly.stl; visual mesh filename=package://assets/urdf_ankle_assembly.stl
- added link urdf_r_upper_femur_assembly, mass 1.912; collision mesh filename=package://assets/r_upper_femur.stl; collision mesh filename=package://assets/stator_x8_p20_120_unified.stl
Joints:
- joint left_ankle_pitch_joint_X4: child udrf_ankle_assembly -> urdf_ankle_assembly
- joint left_ankle_roll_joint_X4: parent udrf_ankle_assembly -> urdf_ankle_assembly
- joint left_knee_joint_X8: limit lower=-1.52716 upper=1.52716 effort=10 velocity=10 -> lower=0 upper=1.51844 effort=10 velocity=10
- joint right_ankle_pitch_joint_X4: child urdf_foot_assembly_2 -> urdf_ankle_assembly_2; origin xyz=-0.012 0.028 -0.004 rpy=0 1.5708 0 -> xyz=0 0.395 0.059 rpy=-0 0 0; parent udrf_ankle_assembly_2 -> urdf_r_tibia_assembly
- joint right_ankle_roll_joint_X4: child udrf_ankle_assembly_2 -> urdf_foot_assembly_2; origin xyz=0 0.395 0.059 rpy=-0 0 0 -> xyz=-0.012 0.028 -0.004 rpy=0 1.5708 0; parent urdf_r_tibia_assembly -> urdf_ankle_assembly_2
- joint right_hip_roll_joint_X8: child urdf_r_upper_femur_assemby -> urdf_r_upper_femur_assembly
- joint right_hip_yaw_joint_X8: parent urdf_r_upper_femur_assemby -> urdf_r_upper_femur_assembly
- joint right_knee_joint_X8: limit lower=-1.52716 upper=1.52716 effort=10 velocity=10 -> lower=0 upper=1.51844 effort=10 velocity=10

File: ldr-harambe-V0.4-com2origin/robot_harambe_v04_com2origin_fixed_axes.urdf (robot description, URDF)
Before this commit: robot robot_harambe_v04_com2origin, 26 links, 25 joints
Links:
- removed link udrf_ankle_assembly
- removed link udrf_ankle_assembly_2
- removed link urdf_r_upper_femur_assemby
- added link urdf_ankle_assembly, mass 0.0818219; collision mesh filename=package://assets/urdf_ankle_assembly.stl; visual mesh filename=package://assets/urdf_ankle_assembly.stl
- added link urdf_ankle_assembly_2, mass 0.0818219; collision mesh filename=package://assets/urdf_ankle_assembly.stl; visual mesh filename=package://assets/urdf_ankle_assembly.stl
- added link urdf_r_upper_femur_assembly, mass 1.912; collision mesh filename=package://assets/r_upper_femur.stl; collision mesh filename=package://assets/stator_x8_p20_120_unified.stl
Joints:
- joint left_ankle_pitch_joint_X4: child udrf_ankle_assembly -> urdf_ankle_assembly
- joint left_ankle_roll_joint_X4: parent udrf_ankle_assembly -> urdf_ankle_assembly
- joint left_knee_joint_X8: limit lower=-1.52716 upper=1.52716 effort=10 velocity=10 -> lower=0 upper=1.51844 effort=10 velocity=10
- joint right_ankle_pitch_joint_X4: axis 1 0 0 -> 0 1 0; child urdf_foot_assembly_2 -> urdf_ankle_assembly_2; origin xyz=-0.012 -0.004 -0.028 rpy=0 0 0 -> xyz=0 0.059 -0.395 rpy=0 0 0; parent udrf_ankle_assembly_2 -> urdf_r_tibia_assembly
- joint right_ankle_roll_joint_X4: axis 0 1 0 -> 1 0 0; child udrf_ankle_assembly_2 -> urdf_foot_assembly_2; origin xyz=0 0.059 -0.395 rpy=0 0 0 -> xyz=-0.012 -0.004 -0.028 rpy=0 0 0; parent urdf_r_tibia_assembly -> urdf_ankle_assembly_2
- joint right_hip_roll_joint_X8: child urdf_r_upper_femur_assemby -> urdf_r_upper_femur_assembly
- joint right_hip_yaw_joint_X8: parent urdf_r_upper_femur_assemby -> urdf_r_upper_femur_assembly
- joint right_knee_joint_X8: limit lower=-1.52716 upper=1.52716 effort=10 velocity=10 -> lower=0 upper=1.51844 effort=10 velocity=10

File: ldr-harambe-V0.4-com2origin/robot_harambe_v04_com2origin_fixed_axes_simplified.urdf (robot description, URDF)
Before this commit: robot robot_harambe_v04_com2origin, 26 links, 25 joints
Links:
- removed link udrf_ankle_assembly
- removed link udrf_ankle_assembly_2
- removed link urdf_r_upper_femur_assemby
- added link urdf_ankle_assembly, mass 0.0818219; collision mesh filename=package://meshes/collision/urdf_ankle_assembly.stl; visual mesh filename=package://meshes/visual/urdf_ankle_assembly.stl
- added link urdf_ankle_assembly_2, mass 0.0818219; collision mesh filename=package://meshes/collision/urdf_ankle_assembly.stl; visual mesh filename=package://meshes/visual/urdf_ankle_assembly.stl
- added link urdf_r_upper_femur_assembly, mass 1.912; collision mesh filename=package://meshes/collision/r_upper_femur.stl; collision mesh filename=package://meshes/collision/stator_x8_p20_120_unified.stl
Joints:
- joint left_ankle_pitch_joint_X4: child udrf_ankle_assembly -> urdf_ankle_assembly
- joint left_ankle_roll_joint_X4: parent udrf_ankle_assembly -> urdf_ankle_assembly
- joint left_knee_joint_X8: limit lower=-1.52716 upper=1.52716 effort=10 velocity=10 -> lower=0 upper=1.51844 effort=10 velocity=10
- joint right_ankle_pitch_joint_X4: axis 1 0 0 -> 0 1 0; child urdf_foot_assembly_2 -> urdf_ankle_assembly_2; origin xyz=-0.012 -0.004 -0.028 rpy=0 0 0 -> xyz=0 0.059 -0.395 rpy=0 0 0; parent udrf_ankle_assembly_2 -> urdf_r_tibia_assembly
- joint right_ankle_roll_joint_X4: axis 0 1 0 -> 1 0 0; child udrf_ankle_assembly_2 -> urdf_foot_assembly_2; origin xyz=0 0.059 -0.395 rpy=0 0 0 -> xyz=-0.012 -0.004 -0.028 rpy=0 0 0; parent urdf_r_tibia_assembly -> urdf_ankle_assembly_2
- joint right_hip_roll_joint_X8: child urdf_r_upper_femur_assemby -> urdf_r_upper_femur_assembly
- joint right_hip_yaw_joint_X8: parent urdf_r_upper_femur_assemby -> urdf_r_upper_femur_assembly
- joint right_knee_joint_X8: limit lower=-1.52716 upper=1.52716 effort=10 velocity=10 -> lower=0 upper=1.51844 effort=10 velocity=10

File: ldr-harambe-V0.4-com2origin/robot_harambe_v04_com2origin_fixed_axes_simplified_no_collision.urdf (robot description, URDF)
Before this commit: robot robot_harambe_v04_com2origin, 26 links, 25 joints
Links:
- removed link udrf_ankle_assembly
- removed link udrf_ankle_assembly_2
- removed link urdf_r_upper_femur_assemby
- added link urdf_ankle_assembly, mass 0.0818219; collision mesh filename=package://meshes/collision/urdf_ankle_assembly.stl; visual mesh filename=package://meshes/visual/urdf_ankle_assembly.stl
- added link urdf_ankle_assembly_2, mass 0.0818219; collision mesh filename=package://meshes/collision/urdf_ankle_assembly.stl; visual mesh filename=package://meshes/visual/urdf_ankle_assembly.stl
- added link urdf_r_upper_femur_assembly, mass 1.912; collision mesh filename=package://meshes/collision/r_upper_femur.stl; visual mesh filename=package://meshes/visual/r_upper_femur.stl
Joints:
- joint left_ankle_pitch_joint_X4: child udrf_ankle_assembly -> urdf_ankle_assembly
- joint left_ankle_roll_joint_X4: parent udrf_ankle_assembly -> urdf_ankle_assembly
- joint left_knee_joint_X8: limit lower=-1.52716 upper=1.52716 effort=10 velocity=10 -> lower=0 upper=1.51844 effort=10 velocity=10
- joint right_ankle_pitch_joint_X4: axis 1 0 0 -> 0 1 0; child urdf_foot_assembly_2 -> urdf_ankle_assembly_2; origin xyz=-0.012 -0.004 -0.028 rpy=0 0 0 -> xyz=0 0.059 -0.395 rpy=0 0 0; parent udrf_ankle_assembly_2 -> urdf_r_tibia_assembly
- joint right_ankle_roll_joint_X4: axis 0 1 0 -> 1 0 0; child udrf_ankle_assembly_2 -> urdf_foot_assembly_2; origin xyz=0 0.059 -0.395 rpy=0 0 0 -> xyz=-0.012 -0.004 -0.028 rpy=0 0 0; parent urdf_r_tibia_assembly -> urdf_ankle_assembly_2
- joint right_hip_roll_joint_X8: child urdf_r_upper_femur_assemby -> urdf_r_upper_femur_assembly
- joint right_hip_yaw_joint_X8: parent urdf_r_upper_femur_assemby -> urdf_r_upper_femur_assembly
- joint right_knee_joint_X8: limit lower=-1.52716 upper=1.52716 effort=10 velocity=10 -> lower=0 upper=1.51844 effort=10 velocity=10

File: ldr-harambe-V0.4-com2origin/urdf/joints/left_foot_joints.xacro (robot description, xacro)
@@ -33,5 +33,5 @@
     <child link="urdf_l_tibia_assembly"/>
     <axis xyz="0 1 0"/>
-    <limit effort="${X8_moderate_effort}" velocity="${X8_rated_velocity}" lower="-1.52716" upper="1.52716"/>
+    <limit effort="${X8_moderate_effort}" velocity="${X8_rated_velocity}" lower="0" upper="1.51844"/>
     <dynamics damping="${X8_damping}" friction="${X8_friction}"/>
   </joint>
@@ -39,5 +39,5 @@
     <origin xyz="0 -0.051 -0.395" rpy="0 0 0"/>
     <parent link="urdf_l_tibia_assembly"/>
-    <child link="udrf_ankle_assembly"/>
+    <child link="urdf_ankle_assembly"/>
     <axis xyz="0 1 0"/>
     <limit effort="${X4_moderate_effort}" velocity="${X4_rated_velocity}" lower="-0.785398" upper="0.785398"/>
@@ -46,5 +46,5 @@
   <joint name="left_ankle_roll_joint_X4" type="${leg_joint_type}">
     <origin xyz="-0.012 -0.004 -0.028" rpy="0 0 0"/>
-    <parent link="udrf_ankle_assembly"/>
+    <parent link="urdf_ankle_assembly"/>
     <child link="urdf_foot_assembly"/>
     <axis xyz="1 0 0"/>

File: ldr-harambe-V0.4-com2origin/urdf/joints/right_foot_joints.xacro (robot description, xacro)
@@ -15,5 +15,5 @@
     <origin xyz="0.053 -0.062 0" rpy="0 0 0"/>
     <parent link="urdf_hip_assembly_2"/>
-    <child link="urdf_r_upper_femur_assemby"/>
+    <child link="urdf_r_upper_femur_assembly"/>
     <axis xyz="1 0 0"/>
     <limit effort="${X8_moderate_effort}" velocity="${X8_rated_velocity}" lower="-3.22886" upper="0.383972"/>
@@ -22,5 +22,5 @@
   <joint name="right_hip_yaw_joint_X8" type="${leg_joint_type}">
     <origin xyz="-0.053 0 -0.217" rpy="0 0 0"/>
-    <parent link="urdf_r_upper_femur_assemby"/>
+    <parent link="urdf_r_upper_femur_assembly"/>
     <child link="urdf_lower_femur_assembly_2"/>
     <axis xyz="0 0 1"/>
@@ -33,18 +33,18 @@
     <child link="urdf_r_tibia_assembly"/>
     <axis xyz="0 1 0"/>
-    <limit effort="${X8_moderate_effort}" velocity="${X8_rated_velocity}" lower="-1.52716" upper="1.52716"/>
+    <limit effort="${X8_moderate_effort}" velocity="${X8_rated_velocity}" lower="0" upper="1.51844"/>
     <dynamics damping="${X8_damping}" friction="${X8_friction}"/>
   </joint>
-  <joint name="right_ankle_roll_joint_X4" type="${leg_joint_type}">
+  <joint name="right_ankle_pitch_joint_X4" type="${leg_joint_type}">
     <origin xyz="0 0.059 -0.395" rpy="0 0 0"/>
     <parent link="urdf_r_tibia_assembly"/>
-    <child link="udrf_ankle_assembly_2"/>
+    <child link="urdf_ankle_assembly_2"/>
     <axis xyz="0 1 0"/>
     <limit effort="${X4_moderate_effort}" velocity="${X4_rated_velocity}" lower="-0.785398" upper="0.785398"/>
     <dynamics damping="${X4_damping}" friction="${X4_friction}"/>
   </joint>
-  <joint name="right_ankle_pitch_joint_X4" type="${leg_joint_type}">
+  <joint name="right_ankle_roll_joint_X4" type="${leg_joint_type}">
     <origin xyz="-0.012 -0.004 -0.028" rpy="0 0 0"/>
-    <parent link="udrf_ankle_assembly_2"/>
+    <parent link="urdf_ankle_assembly_2"/>
     <child link="urdf_foot_assembly_2"/>
     <axis xyz="1 0 0"/>

File: ldr-harambe-V0.4-com2origin/urdf/links/left_foot_links.xacro (robot description, xacro)
@@ -215,5 +215,5 @@
     </collision>
   </link>
-  <link name="udrf_ankle_assembly">
+  <link name="urdf_ankle_assembly">
     <inertial>
       <origin xyz="0 -0.004 -0.0125426" rpy="0 0 0"/>
@@ -224,7 +224,7 @@
       <origin xyz="0 -0.004 -0.0125426" rpy="0 0 -1.5708"/>
       <geometry>
-        <mesh filename="package://full_robot_description/meshes/visual/udrf_ankle_assembly.stl"/>
-      </geometry>
-      <material name="udrf_ankle_assembly_material">
+        <mesh filename="package://full_robot_description/meshes/visual/urdf_ankle_assembly.stl"/>
+      </geometry>
+      <material name="urdf_ankle_assembly_material">
         <color rgba="0.615686 0.811765 0.929412 1"/>
       </material>
@@ -233,5 +233,5 @@
       <origin xyz="0 -0.004 -0.0125426" rpy="0 0 -1.5708"/>
       <geometry>
-        <mesh filename="package://full_robot_description/meshes/collision/udrf_ankle_assembly.stl"/>
+        <mesh filename="package://full_robot_description/meshes/collision/urdf_ankle_assembly.stl"/>
       </geometry>
     </collision>

File: ldr-harambe-V0.4-com2origin/urdf/links/right_foot_links.xacro (robot description, xacro)
@@ -35,5 +35,5 @@
     </visual>
   </link>
-  <link name="urdf_r_upper_femur_assemby">
+  <link name="urdf_r_upper_femur_assembly">
     <inertial>
       <origin xyz="-0.0457109 -0.000406025 -0.147969" rpy="0 0 0"/>
@@ -185,5 +185,5 @@
     </visual>
   </link>
-  <link name="udrf_ankle_assembly_2">
+  <link name="urdf_ankle_assembly_2">
     <inertial>
       <origin xyz="0 -0.004 -0.0125426" rpy="0 0 0"/>
@@ -194,7 +194,7 @@
       <origin xyz="0 -0.004 -0.0125426" rpy="0 0 -1.5708"/>
       <geometry>
-        <mesh filename="package://full_robot_description/meshes/visual/udrf_ankle_assembly.stl"/>
-      </geometry>
-      <material name="udrf_ankle_assembly_2_material">
+        <mesh filename="package://full_robot_description/meshes/visual/urdf_ankle_assembly.stl"/>
+      </geometry>
+      <material name="urdf_ankle_assembly_2_material">
         <color rgba="0.615686 0.811765 0.929412 1"/>
       </material>
@@ -203,5 +203,5 @@
       <origin xyz="0 -0.004 -0.0125426" rpy="0 0 -1.5708"/>
       <geometry>
-        <mesh filename="package://full_robot_description/meshes/collision/udrf_ankle_assembly.stl"/>
+        <mesh filename="package://full_robot_description/meshes/collision/urdf_ankle_assembly.stl"/>
       </geometry>
     </collision>
