Commit message: format com2origin origin2joint

File: ldr-harambe-v0.4-c2o-o2j/robot_harambe_v04_com2origin_origin2joint.urdf (robot description, URDF)
Before this commit: robot robot_harambe_v04_com2origin_origin2joint, 26 links, 25 joints
Links:
- removed link urdf_pelvis
- added link urdf_base, mass 5.778; collision mesh filename=package://assets/urdf_base.stl; visual mesh filename=package://assets/urdf_base.stl
Joints:
- joint left_hip_pitch_joint_X8: parent urdf_pelvis -> urdf_base
- joint right_hip_pitch_joint_X8: parent urdf_pelvis -> urdf_base
- joint waist_yaw_joint_X8: parent urdf_pelvis -> urdf_base
