Commit message: Refactor code structure for improved readability and maintainability

File: ldr-harambe-v0.4-c2o-o2j/robot_harambe_v04_mujoco.urdf (robot description, URDF)
Before this commit: robot robot_harambe_v04_com2origin_origin2joint, 26 links, 25 joints
Links:
- added link world
Joints:
- added joint floating_base: type floating, parent world, child urdf_base
